Commit message: URDF Ackermann update folk

File: AAAckermann/urdf/AAAckermann.urdf (robot description, URDF)
Before this commit: robot AAAckermann, 7 links, 6 joints
Links:
- link base_link: mass 3.70960237040098 -> 5.28323718855656
- link right_steering: mass 0.04056 -> 0.0405602056975407

Commit message: Ackermann URDF update origin

File: AAAckermann/urdf/AAAckermann.urdf (robot description, URDF)
Before this commit: robot AAAckermann, 7 links, 6 joints
Links:
- link base_link: mass 5.28323718855656 -> 5.30323718855656
- link left_steering: mass 0.0405602056975407 -> 0.04056
Joints:
- joint front_left_joint: origin xyz=0.100114914635876 -0.250070257624499 0.198763128382747 rpy=3.14159265358979 0.084917930715728 -1.5707963267949 -> xyz=-0.301000000000045 0.0190000000000679 -0.0695000000000887 rpy=3.14159265358979 0.0849179307157281 -1.5707963267949
- joint front_right_joint: origin xyz=0.661114914635897 -0.250070257624499 0.198763128382747 rpy=3.14159265358979 -0.692237011731428 1.5707963267949 -> xyz=0.259999999999977 0.0190000000000679 -0.0695000000000887 rpy=3.14159265358979 -0.692237011731428 1.5707963267949
- joint left_steering_joint: origin xyz=0.171114914635944 -0.81382025762463 0.184513128382552 rpy=3.14159265358979 0 1.56870378020951 -> xyz=-0.229999999999977 -0.544750000000063 -0.0837500000002837 rpy=3.14159265358979 0 1.56870378020951
- joint right_steering_joint: origin xyz=0.631114914635943 -0.81382025762463 0.184513128382552 rpy=3.14159265358979 0 -1.56162994548732 -> xyz=0.230000000000023 -0.544750000000063 -0.0837500000002836 rpy=3.14159265358979 0 -1.56162994548732

Commit message: URDF ackermann update

File: AAAckermann/urdf/AAAckermann.urdf (robot description, URDF)
Before this commit: robot AAAckermann, 7 links, 6 joints
Links:
- link base_link: mass 5.30323718855656 -> 5.25555128497609
- link left_steering: mass 0.04056 -> 0.0405602056975407
- link right_steering: mass 0.0405602056975407 -> 0.0405602056975408
Joints:
- joint front_left_joint: origin xyz=-0.301000000000045 0.0190000000000679 -0.0695000000000887 rpy=3.14159265358979 0.0849179307157281 -1.5707963267949 -> xyz=0.0190000000000679 0.301000000000045 -0.0695000000000887 rpy=3.14159265358979 0.0849179307157281 3.14159265358979
- joint front_right_joint: origin xyz=0.259999999999977 0.0190000000000679 -0.0695000000000887 rpy=3.14159265358979 -0.692237011731428 1.5707963267949 -> xyz=0.0190000000000679 -0.259999999999977 -0.0695000000000887 rpy=3.14159265358979 -0.692237011731428 0
- joint left_steering_joint: origin xyz=-0.229999999999977 -0.544750000000063 -0.0837500000002837 rpy=3.14159265358979 0 1.56870378020951 -> xyz=-0.544750000000063 0.229999999999977 -0.0837500000002837 rpy=3.14159265358979 0 -0.00209254658538632
- joint right_steering_joint: origin xyz=0.230000000000023 -0.544750000000063 -0.0837500000002836 rpy=3.14159265358979 0 -1.56162994548732 -> xyz=-0.544750000000063 -0.230000000000023 -0.0837500000002836 rpy=3.14159265358979 0 -3.13242627228221
