Commit message: test diff formation

File: my_robot_description/urdf/ackermann_basic.xacro (robot description, xacro)
@@ -1,11 +1,39 @@
 <?xml version="1.0"?>
 <robot xmlns:xacro="http://www.ros.org/wiki/xacro" name="ackermann" >
-  <link name="base_footprint_ack">
-  </link>
-  <joint name="base_link_ack_to_base_footprint_ack" type="fixed">
+  <link name="base_footprint">
+  </link>
+  <joint name="base_link_to_base_footprint" type="fixed">
     <origin xyz="0 0 0.12" rpy="0 0 0"/>
-    <parent link="base_footprint_ack"/>
+    <parent link="base_footprint"/>
     <child link="base_link"/>
   </joint>
+  <link name="laser_frame">
+    <visual>
+      <geometry>
+        <cylinder radius="0.05" length="0.04"/>
+      </geometry>
+    </visual>
+    <collision>
+      <geometry>
+        <cylinder radius="0.05" length="0.04"/>
+      </geometry>
+    </collision>
+    <inertial>
+      <origin
+        xyz="0 0 0"
+        rpy="0 0 0" />
+      <mass
+        value="0.01" />
+      <inertia
+        ixx="0.01" ixy="0.0" ixz="0.0"
+        iyy="0.01" iyz="0.0"
+        izz="0.01"/>
+    </inertial>
+  </link>
+  <joint name="laser_joint" type="fixed">
+    <origin xyz="0 0 0.12" rpy="0 0 0"/>
+    <parent link="base_link"/>
+    <child link="laser_frame"/>
+  </joint>
   <link
     name="base_link">
@@ -15,12 +43,9 @@
         rpy="0 0 0" />
       <mass
-        value="1.25555128497609" />
-      <inertia
-        ixx="0.0414328478617682"
-        ixy="-1.82796488685318E-07"
-        ixz="3.45960820664179E-07"
-        iyy="0.0417152661425413"
-        iyz="1.05010040923958E-07"
-        izz="0.0821338918053197" />
+        value="0.525555128497609" />
+      <inertia
+        ixx="0.01" ixy="0.0" ixz="0.0"
+        iyy="0.01" iyz="0.0"
+        izz="0.01"/>
     </inertial>
     <visual>
@@ -55,12 +80,9 @@
         rpy="0 0 0" />
       <mass
-        value="0.24047" />
-      <inertia
-        ixx="0.00024514"
-        ixy="5.4339E-21"
-        ixz="-6.7763E-21"
-        iyy="0.00045262"
-        iyz="6.4709E-20"
-        izz="0.00024514" />
+        value="2.4" />
+      <inertia
+        ixx="0.01" ixy="0.0" ixz="0.0"
+        iyy="0.01" iyz="0.0"
+        izz="0.01"/>
     </inertial>
     <visual>
@@ -90,5 +112,5 @@
   <joint
     name="front_left_joint"
-    type="continuous">
+    type="fixed">
     <origin
       xyz="0.0190000000000679 0.301000000000045 -0.0695000000000887"
@@ -108,12 +130,9 @@
         rpy="0 0 0" />
       <mass
-        value="0.24047" />
-      <inertia
-        ixx="0.00024514"
-        ixy="5.2554E-21"
-        ixz="0"
-        iyy="0.00045262"
-        iyz="4.3994E-20"
-        izz="0.00024514" />
+        value="2.4" />
+      <inertia
+        ixx="0.01" ixy="0.0" ixz="0.0"
+        iyy="0.01" iyz="0.0"
+        izz="0.01"/>
     </inertial>
     <visual>
@@ -143,5 +162,5 @@
   <joint
     name="front_right_joint"
-    type="continuous">
+    type="fixed">
     <origin
       xyz="0.0190000000000679 -0.259999999999977 -0.0695000000000887"
@@ -163,10 +182,7 @@
         value="0.0405602056975407" />
       <inertia
-        ixx="1.43958495481578E-05"
-        ixy="-1.73339990683825E-06"
-        ixz="-7.11935154287877E-06"
-        iyy="2.95171085845272E-05"
-        iyz="2.08772590818048E-06"
-        izz="3.10994722329793E-05" />
+        ixx="0.01" ixy="0.0" ixz="0.0"
+        iyy="0.01" iyz="0.0"
+        izz="0.01"/>
     </inertial>
     <visual>
@@ -196,5 +212,5 @@
   <joint
     name="left_steering_joint"
-    type="continuous">
+    type="fixed">
     <origin
       xyz="-0.544750000000063 0.229999999999977 -0.0837500000002837"
@@ -214,12 +230,9 @@
         rpy="0 0 0" />
       <mass
-        value="0.24047" />
-      <inertia
-        ixx="0.00024514"
-        ixy="-4.9967E-09"
-        ixz="-5.3615E-10"
-        iyy="0.00045026"
-        iyz="2.201E-05"
-        izz="0.0002475" />
+        value="2.4" />
+      <inertia
+        ixx="0.01" ixy="0.0" ixz="0.0"
+        iyy="0.01" iyz="0.0"
+        izz="0.01"/>
     </inertial>
     <visual>
@@ -249,5 +262,5 @@
   <joint
     name="rear_left_joint"
-    type="continuous">
+    type="fixed">
     <origin
       xyz="0 -0.0367488381424265 -0.0159999999999999"
@@ -269,10 +282,7 @@
         value="0.0405602056975408" />
       <inertia
-        ixx="1.49389187707206E-05"
-        ixy="3.30295116006257E-06"
-        ixz="7.3015684371967E-06"
-        iyy="2.89780797923847E-05"
-        iyz="1.31491150207248E-06"
-        izz="3.11035126633983E-05" />
+        ixx="0.01" ixy="0.0" ixz="0.0"
+        iyy="0.01" iyz="0.0"
+        izz="0.01"/>
     </inertial>
     <visual>
@@ -302,5 +312,5 @@
   <joint
     name="right_steering_joint"
-    type="continuous">
+    type="fixed">
     <origin
       xyz="-0.544750000000063 -0.230000000000023 -0.0837500000002836"
@@ -320,12 +330,9 @@
         rpy="0 0 0" />
       <mass
-        value="0.24047" />
-      <inertia
-        ixx="0.00024514"
-        ixy="4.6696E-13"
-        ixz="9.4021E-20"
-        iyy="0.00045262"
-        iyz="4.2319E-11"
-        izz="0.00024514" />
+        value="2.4" />
+      <inertia
+        ixx="0.01" ixy="0.0" ixz="0.0"
+        iyy="0.01" iyz="0.0"
+        izz="0.01"/>
     </inertial>
     <visual>
@@ -355,5 +362,5 @@
   <joint
     name="rear_right_joint"
-    type="continuous">
+    type="fixed">
     <origin
       xyz="0 -0.0370034448281129 -0.0159999999999995"
@@ -366,48 +373,55 @@
       xyz="0 1 0" />
   </joint>
- <gazebo>
-    <plugin name="gazebo_ros_ackermann_drive" filename="libgazebo_ros_ackermann_drive.so">
+  <gazebo>
+    <plugin name="gazebo_ros_planar_move_ack" filename="libgazebo_ros_planar_move.so">
       <ros>
-        <namespace>/ackermann</namespace>
+        <!-- Add a namespace -->
+        <namespace></namespace>
+        <!-- Remap the default topic -->
+        <remapping>/cmd_vel:=/cmd_vel</remapping>
+        <remapping>odom:=/diffdrive/odom</remapping>
       </ros>
-      <update_rate>100.0</update_rate>
-      <wheel_base>0.65</wheel_base>
-      <wheel_separation>0.55</wheel_separation>
-      <wheel_radius>0.06</wheel_radius>
-      <!-- wheels -->
-      <front_left_joint>rear_right_joint</front_left_joint>
-      <front_right_joint>rear_left_joint</front_right_joint>
-      <rear_left_joint>front_right_joint</rear_left_joint>
-      <rear_right_joint>front_left_joint</rear_right_joint>
-      <!-- wheels -->
-      <!-- <front_left_joint>front_left_joint</front_left_joint>
-      <front_right_joint>front_right_joint</front_right_joint>
-      <rear_left_joint>rear_left_joint</rear_left_joint>
-      <rear_right_joint>rear_right_joint</rear_right_joint> -->
-      <!-- steering joints -->
-      <left_steering_joint>right_steering_joint</left_steering_joint>
-      <right_steering_joint>left_steering_joint</right_steering_joint>
-      <!-- Max absolute steer angle for tyre in radians-->
-      <!-- Any cmd_vel angular z greater than this would be capped -->
-      <max_steer>0.6458</max_steer>
-      <!-- Max absolute steering angle of steering wheel -->
-      <max_steering_angle>7.85</max_steering_angle>
-      <!-- Max absolute linear speed in m/s -->
-      <max_speed>20</max_speed>
-      <!-- PID tuning -->
-      <left_steering_pid_gain>1 0 1</left_steering_pid_gain>
-      <left_steering_i_range>0 0</left_steering_i_range>
-      <right_steering_pid_gain>1 0 1</right_steering_pid_gain>
-      <right_steering_i_range>0 0</right_steering_i_range>
-      <linear_velocity_pid_gain>1000 0 1</linear_velocity_pid_gain>
-      <linear_velocity_i_range>0 0</linear_velocity_i_range>
+      <update_rate>50</update_rate>
+      <publish_rate>50</publish_rate>
       <!-- output -->
       <publish_odom>true</publish_odom>
       <publish_odom_tf>true</publish_odom_tf>
+      <odometry_frame>odom</odometry_frame>
+      <robot_base_frame>base_footprint</robot_base_frame>
       <publish_wheel_tf>true</publish_wheel_tf>
-      <publish_distance>true</publish_distance>
-      <odometry_frame>odom_ack</odometry_frame>
-      <robot_base_frame>base_link</robot_base_frame>
+      <covariance_x>0.0001</covariance_x>
+      <covariance_y>0.0001</covariance_y>
+      <covariance_yaw>0.01</covariance_yaw>
     </plugin>
   </gazebo>
+ <gazebo reference="laser_frame">
+    <material>Gazebo/Orange</material>
+    <sensor name="laser" type="ray">
+      <namespace></namespace>
+      <pose>0 0 0 0 0 0</pose>
+      <visualize>false</visualize>
+      <update_rate>10</update_rate>
+      <ray>
+        <scan>
+          <horizontal>
+            <samples>360</samples>
+            <min_angle>-3.14</min_angle>
+            <max_angle>3.14</max_angle>
+          </horizontal>
+        </scan>
+        <range>
+          <min>0.3</min>
+          <max>12</max>
+        </range>
+      </ray>
+      <plugin name="laser" filename="libgazebo_ros_ray_sensor.so">
+        <namespace></namespace>
+        <ros>
+          <argument>~/out:=scan</argument>
+        </ros>
+        <output_type>sensor_msgs/LaserScan</output_type>
+        <frame_name>laser_frame</frame_name>
+      </plugin>
+    </sensor>
+  </gazebo>
 </robot>

File: my_robot_description/urdf/diffdrive.xacro (robot description, xacro)
@@ -6,11 +6,11 @@
   <material name="wheel">
     <color rgba="0 1 0 0.5" /> </material>
-  <link name="base_footprint"></link>
-  <joint name="base_link_to_base_footprint" type="fixed">
-    <origin xyz="0 0 0" rpy="0 0 0"/>
-    <parent link="base_footprint"/>
-    <child link="base_link"/>
-  </joint>
-  <link name="laser_frame">
+  <link name="base_footprint_diff"></link>
+  <joint name="base_link_diff_to_base_footprint_diff" type="fixed">
+    <origin xyz="0 0 0" rpy="0 0 3.14159265"/>
+    <parent link="base_footprint_diff"/>
+    <child link="base_link_diff"/>
+  </joint>
+  <link name="laser_frame_diff">
     <visual>
       <geometry>
@@ -36,10 +36,10 @@
   </link>
   <joint name="laser_joint" type="fixed">
-    <origin xyz="0 0 0.12" rpy="0 0 0"/>
-    <parent link="base_link"/>
-    <child link="laser_frame"/>
+    <origin xyz="0 0 0.22" rpy="0 0 0"/>
+    <parent link="base_link_diff"/>
+    <child link="laser_frame_diff"/>
   </joint>
   <link
-    name="base_link">
+    name="base_link_diff">
     <inertial>
       <origin
@@ -117,5 +117,5 @@
   </link>
   <joint
-    name="right_wheel_joint"
+    name="left_wheel_joint"
     type="continuous">
     <origin
@@ -123,9 +123,9 @@
       rpy="0 0.774914173734372 3.14159265358979" />
     <parent
-      link="base_link" />
+      link="base_link_diff" />
     <child
       link="wheel_left" />
     <axis
-      xyz="0 -1 0" />
+      xyz="0 1 0" />
   </joint>
   <link
@@ -166,5 +166,5 @@
   </link>
   <joint
-    name="left_wheel_joint"
+    name="right_wheel_joint"
     type="continuous">
     <origin
@@ -172,9 +172,9 @@
       rpy="3.14159265358979 -0.53712555837446 3.14159265358979" />
     <parent
-      link="base_link" />
+      link="base_link_diff" />
     <child
       link="wheel_right" />
     <axis
-      xyz="0 1 0" />
+      xyz="0 -1 0" />
   </joint>
     <gazebo>
@@ -183,5 +183,6 @@
             <ros>
             <!-- Add a namespace -->
-            <namespace></namespace>
+            <namespace>diff</namespace>
+             <remapping>/diff/cmd_vel:=/cmd_vel_follower</remapping>
             </ros>
             <update_rate>50</update_rate>
@@ -193,5 +194,5 @@
             <wheel_diameter>0.12</wheel_diameter>
             <!-- input -->
-            <command_topic>cmd_vel</command_topic>
+            <command_topic>cmd_vel_follower</command_topic>
             <!-- output -->
             <publish_odom>true</publish_odom>
@@ -201,9 +202,9 @@
             <publish_wheel_tf>true</publish_wheel_tf>
             <odometry_topic>diffdrive/odom</odometry_topic>
-            <odometry_frame>odom</odometry_frame>
-            <robot_base_frame>base_footprint</robot_base_frame>
+            <odometry_frame>diff_odom</odometry_frame>
+            <robot_base_frame>base_footprint_diff</robot_base_frame>
         </plugin>
     </gazebo>
-    <gazebo reference="laser_frame">
+    <gazebo reference="laser_frame_diff">
         <material>Gazebo/Red</material>
         <sensor name="laser" type="ray">
@@ -224,10 +225,10 @@
                 </range>
             </ray>
-            <plugin name="laser_controller" filename="libgazebo_ros_ray_sensor.so">
+            <plugin name="laser_controller_diff" filename="libgazebo_ros_ray_sensor.so">
                 <ros>
-                    <argument>~/out:=scan</argument>
+                    <argument>~/out:=scan_diff</argument>
                 </ros>
                 <output_type>sensor_msgs/LaserScan</output_type>
-                <frame_name>laser_frame</frame_name>
+                <frame_name>laser_frame_diff</frame_name>
             </plugin>
         </sensor>

File: my_robot_description/urdf/long_pallet.xacro (robot description, xacro)
@@ -1,18 +1,23 @@
-<?xml version="1.0"?>
-<robot name="long_pallet" xmlns:xacro="http://www.ros.org/wiki/xacro">
-  <link name="long_pallet">
+<?xml version="1.0" encoding="utf-8"?>
+<robot xmlns:xacro="http://www.ros.org/wiki/xacro" name="long_pallet">
+  <link name="pallet_footprint">
+  </link>
+  <joint name="pallet_link_to_pallet_footprint" type="fixed">
+    <origin xyz="0 0 0" rpy="0 0 0"/>
+    <parent link="pallet_footprint"/>
+    <child link="pallet_link"/>
+  </joint>
+  <link
+    name="pallet_link">
     <inertial>
       <origin
-        xyz="0.291080013901068 0.20335853380665 0.313229331004487"
+        xyz="0 0 0"
         rpy="0 0 0" />
       <mass
-        value="5.89400000000001" />
+        value="1000" />
       <inertia
-        ixx="0.122033819833333"
-        ixy="-1.88845020711894E-20"
-        ixz="-1.53871349224279E-17"
-        iyy="0.157871233333333"
-        iyz="-4.14514250944756E-20"
-        izz="0.0361096948333333" />
+        ixx="0.01" ixy="0.0" ixz="0.0"
+        iyy="0.01" iyz="0.0"
+        izz="0.01"/>
     </inertial>
     <visual>
@@ -22,6 +27,5 @@
       <geometry>
         <mesh
-          filename="file:///$(find my_robot_description)/meshes/long_pallet.stl">
-        </mesh>
+          filename="file:///$(find my_robot_description)/meshes/pallet/base_link.STL" />
       </geometry>
       <material
@@ -37,22 +41,7 @@
       <geometry>
         <mesh
-          filename="file:///$(find my_robot_description)/meshes/long_pallet.stl">
-        </mesh>
+          filename="file:///$(find my_robot_description)/meshes/pallet/base_link.STL" />
       </geometry>
     </collision>
   </link>
-  <link name="base_footprint">
-      <origin xyz="0 0 0" rpy="0 0 0" />
-  </link>
-  <joint name="base_joint" type="fixed">
-      <parent link="base_footprint"/>
-      <child link="long_pallet"/>
-      <origin xyz="0 0 0" rpy="0 0 0" />
-  </joint>
-  <!-- <gazebo>
-      <plugin name="gazebo_ros_joint_state_publisher_pallet"
-          filename="libgazebo_ros_joint_state_publisher.so">
-          <joint_name>base_joint</joint_name>
-      </plugin>
-  </gazebo> -->
 </robot>

Commit message: re-organized

File: my_robot_description/urdf/ackermann_basic.xacro (robot description, xacro)
@@ -32,5 +32,5 @@
   </link>
   <joint name="laser_joint" type="fixed">
-    <origin xyz="0 0 0.12" rpy="0 0 0"/>
+    <origin xyz="0 0 0.08" rpy="0 0 0"/>
     <parent link="base_link"/>
     <child link="laser_frame"/>
@@ -43,9 +43,12 @@
         rpy="0 0 0" />
       <mass
-        value="0.525555128497609" />
-      <inertia
-        ixx="0.01" ixy="0.0" ixz="0.0"
-        iyy="0.01" iyz="0.0"
-        izz="0.01"/>
+        value="5.25555128497609" />
+      <inertia
+        ixx="0.0414328478617682"
+        ixy="-1.82796488685318E-07"
+        ixz="3.45960820664179E-07"
+        iyy="0.0417152661425413"
+        iyz="1.05010040923958E-07"
+        izz="0.0821338918053197" />
     </inertial>
     <visual>
@@ -71,4 +74,12 @@
           filename="file:///$(find my_robot_description)/meshes/ackermann_meshes/base_link.STL" />
       </geometry>
+      <surface>
+        <friction>
+          <ode>
+            <mu>0.001</mu>
+            <mu2>0.001</mu2>
+          </ode>
+        </friction>
+      </surface>
     </collision>
   </link>
@@ -82,7 +93,10 @@
         value="2.4" />
       <inertia
-        ixx="0.01" ixy="0.0" ixz="0.0"
-        iyy="0.01" iyz="0.0"
-        izz="0.01"/>
+        ixx="0.00024514"
+        ixy="5.4339E-21"
+        ixz="-6.7763E-21"
+        iyy="0.00045262"
+        iyz="6.4709E-20"
+        izz="0.00024514" />
     </inertial>
     <visual>
@@ -132,7 +146,10 @@
         value="2.4" />
       <inertia
-        ixx="0.01" ixy="0.0" ixz="0.0"
-        iyy="0.01" iyz="0.0"
-        izz="0.01"/>
+        ixx="0.00024514"
+        ixy="5.2554E-21"
+        ixz="0"
+        iyy="0.00045262"
+        iyz="4.3994E-20"
+        izz="0.00024514" />
     </inertial>
     <visual>
@@ -180,9 +197,12 @@
         rpy="0 0 0" />
       <mass
-        value="0.0405602056975407" />
-      <inertia
-        ixx="0.01" ixy="0.0" ixz="0.0"
-        iyy="0.01" iyz="0.0"
-        izz="0.01"/>
+        value="4" />
+      <inertia
+        ixx="1.43958495481578E-05"
+        ixy="-1.73339990683825E-06"
+        ixz="-7.11935154287877E-06"
+        iyy="2.95171085845272E-05"
+        iyz="2.08772590818048E-06"
+        izz="3.10994722329793E-05" />
     </inertial>
     <visual>
@@ -232,7 +252,10 @@
         value="2.4" />
       <inertia
-        ixx="0.01" ixy="0.0" ixz="0.0"
-        iyy="0.01" iyz="0.0"
-        izz="0.01"/>
+        ixx="0.00024514"
+        ixy="-4.9967E-09"
+        ixz="-5.3615E-10"
+        iyy="0.00045026"
+        iyz="2.201E-05"
+        izz="0.0002475" />
     </inertial>
     <visual>
@@ -280,9 +303,12 @@
         rpy="0 0 0" />
       <mass
-        value="0.0405602056975408" />
-      <inertia
-        ixx="0.01" ixy="0.0" ixz="0.0"
-        iyy="0.01" iyz="0.0"
-        izz="0.01"/>
+        value="4" />
+      <inertia
+        ixx="1.49389187707206E-05"
+        ixy="3.30295116006257E-06"
+        ixz="7.3015684371967E-06"
+        iyy="2.89780797923847E-05"
+        iyz="1.31491150207248E-06"
+        izz="3.11035126633983E-05" />
     </inertial>
     <visual>
@@ -332,7 +358,10 @@
         value="2.4" />
       <inertia
-        ixx="0.01" ixy="0.0" ixz="0.0"
-        iyy="0.01" iyz="0.0"
-        izz="0.01"/>
+        ixx="0.00024514"
+        ixy="4.6696E-13"
+        ixz="9.4021E-20"
+        iyy="0.00045262"
+        iyz="4.2319E-11"
+        izz="0.00024514" />
     </inertial>
     <visual>
@@ -373,4 +402,22 @@
       xyz="0 1 0" />
   </joint>
+    <gazebo reference="front_left">
+      <material>Gazebo/Green</material>
+    </gazebo>
+    <gazebo reference="front_right">
+      <material>Gazebo/Green</material>
+    </gazebo>
+    <gazebo reference="rear_left">
+      <material>Gazebo/Green</material>
+    </gazebo>
+    <gazebo reference="rear_right">
+      <material>Gazebo/Green</material>
+    </gazebo>
+    <gazebo reference="right_steering">
+      <material>Gazebo/Red</material>
+    </gazebo>
+    <gazebo reference="left_steering">
+      <material>Gazebo/Red</material>
+    </gazebo>
   <gazebo>
     <plugin name="gazebo_ros_planar_move_ack" filename="libgazebo_ros_planar_move.so">
@@ -382,6 +429,6 @@
         <remapping>odom:=/diffdrive/odom</remapping>
       </ros>
-      <update_rate>50</update_rate>
-      <publish_rate>50</publish_rate>
+      <update_rate>100</update_rate>
+      <publish_rate>100</publish_rate>
       <!-- output -->
       <publish_odom>true</publish_odom>
@@ -390,11 +437,12 @@
       <robot_base_frame>base_footprint</robot_base_frame>
       <publish_wheel_tf>true</publish_wheel_tf>
+<!--
       <covariance_x>0.0001</covariance_x>
       <covariance_y>0.0001</covariance_y>
-      <covariance_yaw>0.01</covariance_yaw>
+      <covariance_yaw>0.01</covariance_yaw> -->
     </plugin>
   </gazebo>
  <gazebo reference="laser_frame">
-    <material>Gazebo/Orange</material>
+    <material>Gazebo/Black</material>
     <sensor name="laser" type="ray">
       <namespace></namespace>

File: my_robot_description/urdf/diffdrive.xacro (robot description, xacro)
@@ -36,5 +36,5 @@
   </link>
   <joint name="laser_joint" type="fixed">
-    <origin xyz="0 0 0.22" rpy="0 0 0"/>
+    <origin xyz="0 0 0.12" rpy="0 0 0"/>
     <parent link="base_link_diff"/>
     <child link="laser_frame_diff"/>
@@ -78,4 +78,12 @@
           filename="file:///$(find my_robot_description)/meshes/diffdrive_meshes/base_link.STL" />
       </geometry>
+      <surface>
+        <friction>
+          <ode>
+            <mu>0.001</mu>
+            <mu2>0.001</mu2>
+          </ode>
+        </friction>
+      </surface>
     </collision>
   </link>
@@ -206,6 +214,15 @@
         </plugin>
     </gazebo>
+    <gazebo reference="wheel_right">
+      <material>Gazebo/Green</material>
+    </gazebo>
+    <gazebo reference="wheel_left">
+      <material>Gazebo/Green</material>
+    </gazebo>
+    <gazebo reference="base_link_diff">
+      <material>Gazebo/White</material>
+    </gazebo>
     <gazebo reference="laser_frame_diff">
-        <material>Gazebo/Red</material>
+        <material>Gazebo/Black</material>
         <sensor name="laser" type="ray">
             <pose> 0 0 0 0 0 0 </pose>

File: my_robot_description/urdf/long_pallet.xacro (robot description, xacro)
@@ -12,12 +12,15 @@
     <inertial>
       <origin
-        xyz="0 0 0"
+        xyz="2.22044604925031E-16 2.22044604925031E-16 0.0802779743476336"
         rpy="0 0 0" />
       <mass
-        value="1000" />
+        value="1" />
       <inertia
-        ixx="0.01" ixy="0.0" ixz="0.0"
-        iyy="0.01" iyz="0.0"
-        izz="0.01"/>
+        ixx="0.05011773"
+        ixy="3.14732432919024E-18"
+        ixz="6.18375078595321E-17"
+        iyy="0.556581597187501"
+        iyz="4.10639232657203E-20"
+        izz="0.602756250000001" />
     </inertial>
     <visual>
@@ -43,5 +46,19 @@
           filename="file:///$(find my_robot_description)/meshes/pallet/base_link.STL" />
       </geometry>
+      <surface>
+        <friction>
+          <ode>
+            <mu>0.001</mu>
+            <mu2>0.001</mu2>
+          </ode>
+        </friction>
+      </surface>
     </collision>
   </link>
+  <material name="verylightbrown" >
+    <color rgba="0.8274509803921568 0.7137254901960784 0.5137254901960784 1.0" />
+  </material>
+  <gazebo reference="pallet_link">
+      <material>Gazebo/Wood</material>
+  </gazebo>
 </robot>

File: my_robot_description/urdf/world.xacro (robot description, xacro)
@@ -45,3 +45,6 @@
     </collision>
   </link>
+  <gazebo reference="map_link">
+      <material>Gazebo/Black</material>
+  </gazebo>
 </robot>
