Commit message: edit topic name

File: my_robot_description/urdf/ackermann_basic.xacro (robot description, xacro)
@@ -75,8 +75,21 @@
       </geometry>
       <surface>
+        <contact>
+          <poissons_ratio>0.347</poissons_ratio>
+          <elastic_modulus>8.8e+09</elastic_modulus>
+          <ode>
+            <soft_cfm>0.0</soft_cfm>
+            <soft_erp>0.2</soft_erp>
+            <kp>1e25</kp>
+            <kd>1e13</kd>
+            <max_vel>0.01</max_vel>
+            <min_depth>0.0001</min_depth>
+          </ode>
+        </contact>
         <friction>
           <ode>
-            <mu>0.001</mu>
-            <mu2>0.001</mu2>
+            <mu>0.1</mu>
+            <mu2>0.1</mu2>
+        <fdir1>1 0 0</fdir1>
           </ode>
         </friction>

File: my_robot_description/urdf/diffdrive.xacro (robot description, xacro)
@@ -79,8 +79,21 @@
       </geometry>
       <surface>
+        <contact>
+          <poissons_ratio>0.347</poissons_ratio>
+          <elastic_modulus>8.8e+09</elastic_modulus>
+          <ode>
+            <soft_cfm>0.0</soft_cfm>
+            <soft_erp>0.2</soft_erp>
+            <kp>1e25</kp>
+            <kd>1e13</kd>
+            <max_vel>0.01</max_vel>
+            <min_depth>0.0001</min_depth>
+          </ode>
+        </contact>
         <friction>
           <ode>
-            <mu>0.001</mu>
-            <mu2>0.001</mu2>
+            <mu>0.1</mu>
+            <mu2>0.1</mu2>
+        <fdir1>1 0 0</fdir1>
           </ode>
         </friction>

File: my_robot_description/urdf/long_pallet.xacro (robot description, xacro)
@@ -15,5 +15,5 @@
         rpy="0 0 0" />
       <mass
-        value="1" />
+        value="0.1" />
       <inertia
         ixx="0.05011773"
@@ -47,8 +47,21 @@
       </geometry>
       <surface>
+        <contact>
+          <poissons_ratio>0.347</poissons_ratio>
+          <elastic_modulus>8.8e+09</elastic_modulus>
+          <ode>
+            <soft_cfm>0.0</soft_cfm>
+            <soft_erp>0.2</soft_erp>
+            <kp>1e25</kp>
+            <kd>1e13</kd>
+            <max_vel>0.01</max_vel>
+            <min_depth>0.0001</min_depth>
+          </ode>
+        </contact>
         <friction>
           <ode>
-            <mu>0.001</mu>
-            <mu2>0.001</mu2>
+            <mu>1000</mu>
+            <mu2>1000</mu2>
+        <fdir1>1 0 0</fdir1>
           </ode>
         </friction>

File: my_robot_description/urdf/mecanum.xacro (robot description, xacro)
@@ -43,9 +43,12 @@
         rpy="0 0 0" />
       <mass
-        value="0.5" />
-      <inertia
-        ixx="0.01" ixy="0.0" ixz="0.0"
-        iyy="0.01" iyz="0.0"
-        izz="0.01"/>
+        value="5" />
+      <inertia
+        ixx="0.0576995775576278"
+        ixy="5.10236521313111E-19"
+        ixz="-5.64437487412692E-14"
+        iyy="0.0133526650283985"
+        iyz="-4.8820083846232E-08"
+        izz="0.0706132037943649" />
     </inertial>
     <visual>
@@ -80,5 +83,5 @@
         rpy="0 0 0" />
       <mass
-        value="0.0002" />
+        value="2.1" />
       <inertia
         ixx="0.01" ixy="0.0" ixz="0.0"
@@ -113,6 +116,6 @@
     type="fixed">
     <origin
-      xyz="0.196431540449915 0.18250000000009 -0.0500000000000465"
-      rpy="2.56826265176299 -0.701812030330357 2.7542816171153" />
+      xyz="0.195390712673452 0.172500000000024 -0.0850000000000468"
+      rpy="1.5707963267949 0 1.5707963267949" />
     <parent
       link="base_link_mec" />
@@ -120,5 +123,5 @@
       link="wheel_fr_right" />
     <axis
-      xyz="0.707106781183754 -0.64156167526822 0.297319048886856" />
+      xyz="0 0 -1" />
   </joint>
   <link
@@ -129,5 +132,5 @@
         rpy="0 0 0" />
       <mass
-        value="0.0002" />
+        value="2.1" />
       <inertia
         ixx="0.01" ixy="0.0" ixz="0.0"
@@ -162,6 +165,6 @@
     type="fixed">
     <origin
-      xyz="0.196431540449915 -0.182499999999932 -0.0500000000000465"
-      rpy="2.56826265176299 -0.701812030330358 2.7542816171153" />
+      xyz="0.195390712673452 -0.192499999999931 -0.0850000000000466"
+      rpy="-1.5707963267949 0 -1.5707963267949" />
     <parent
       link="base_link_mec" />
@@ -169,5 +172,5 @@
       link="wheel_bk_right" />
     <axis
-      xyz="0.707106781183753 -0.641561675268222 0.297319048886854" />
+      xyz="0 0 -1" />
   </joint>
   <link
@@ -178,5 +181,5 @@
         rpy="0 0 0" />
       <mass
-        value="0.0002" />
+        value="2.1" />
       <inertia
         ixx="0.01" ixy="0.0" ixz="0.0"
@@ -211,6 +214,6 @@
     type="fixed">
     <origin
-      xyz="-0.141459172223538 0.18250000000009 -0.0500000000000464"
-      rpy="2.56826265176299 -0.701812030330358 2.7542816171153" />
+      xyz="-0.195390712673501 0.172500000000024 -0.085000000000046"
+      rpy="1.5707963267949 0 -1.5707963267949" />
     <parent
       link="base_link_mec" />
@@ -218,5 +221,5 @@
       link="wheel_fr_left" />
     <axis
-      xyz="0.707106781183754 -0.641561675268221 0.297319048886855" />
+      xyz="0 0 1" />
   </joint>
   <link
@@ -227,5 +230,5 @@
         rpy="0 0 0" />
       <mass
-        value="0.0002" />
+        value="2.1" />
       <inertia
         ixx="0.01" ixy="0.0" ixz="0.0"
@@ -260,6 +263,6 @@
     type="fixed">
     <origin
-      xyz="-0.141459172223538 -0.182499999999932 -0.0500000000000464"
-      rpy="2.56826265176298 -0.701812030330358 2.7542816171153" />
+      xyz="-0.195390712673501 -0.192499999999931 -0.085000000000046"
+      rpy="1.5707963267949 0 -1.5707963267949" />
     <parent
       link="base_link_mec" />
@@ -267,6 +270,18 @@
       link="wheel_bk_left" />
     <axis
-      xyz="0.707106781183753 -0.641561675268222 0.297319048886854" />
-  </joint>
+      xyz="0 0 1" />
+  </joint>
+    <gazebo reference="wheel_fr_left">
+      <material>Gazebo/Grey</material>
+    </gazebo>
+    <gazebo reference="wheel_fr_right">
+      <material>Gazebo/Grey</material>
+    </gazebo>
+    <gazebo reference="wheel_bk_left">
+      <material>Gazebo/Grey</material>
+    </gazebo>
+    <gazebo reference="wheel_bk_right">
+      <material>Gazebo/Grey</material>
+    </gazebo>
 <gazebo>
   <plugin name="gazebo_ros_planar_move" filename="libgazebo_ros_planar_move.so">

Commit message: diffdrive_control

File: my_robot_description/urdf/ackermann_basic.xacro (robot description, xacro)
@@ -74,25 +74,4 @@
           filename="file:///$(find my_robot_description)/meshes/ackermann_meshes/base_link.STL" />
       </geometry>
-      <surface>
-        <contact>
-          <poissons_ratio>0.347</poissons_ratio>
-          <elastic_modulus>8.8e+09</elastic_modulus>
-          <ode>
-            <soft_cfm>0.0</soft_cfm>
-            <soft_erp>0.2</soft_erp>
-            <kp>1e25</kp>
-            <kd>1e13</kd>
-            <max_vel>0.01</max_vel>
-            <min_depth>0.0001</min_depth>
-          </ode>
-        </contact>
-        <friction>
-          <ode>
-            <mu>0.1</mu>
-            <mu2>0.1</mu2>
-        <fdir1>1 0 0</fdir1>
-          </ode>
-        </friction>
-      </surface>
     </collision>
   </link>
@@ -210,5 +189,5 @@
         rpy="0 0 0" />
       <mass
-        value="4" />
+        value="2" />
       <inertia
         ixx="1.43958495481578E-05"
@@ -316,5 +295,5 @@
         rpy="0 0 0" />
       <mass
-        value="4" />
+        value="2" />
       <inertia
         ixx="1.49389187707206E-05"

File: my_robot_description/urdf/diffdrive_control.xacro (robot description, xacro)
@@ -178,32 +178,42 @@
       xyz="0 -1 0" />
   </joint>
-    <gazebo>
-        <plugin name="gazebo_ros_diff_drive" filename="libgazebo_ros_diff_drive.so">
-            <!-- Update rate in Hz -->
-            <ros>
-            <!-- Add a namespace -->
-            <namespace>diff</namespace>
-             <remapping>/diff/cmd_vel:=/cmd_vel_follower</remapping>
-            </ros>
-            <update_rate>50</update_rate>
-            <!-- wheels -->
-            <left_joint>left_wheel_joint</left_joint>
-            <right_joint>right_wheel_joint</right_joint>
-            <!-- kinematics -->
-            <wheel_separation>0.5</wheel_separation>
-            <wheel_diameter>0.12</wheel_diameter>
-            <!-- input -->
-            <command_topic>cmd_vel_follower</command_topic>
-            <!-- output -->
-            <publish_odom>true</publish_odom>
-            <!-- Odometry source, 0 for ENCODER, 1 for WORLD, defaults to WORLD -->
-            <odometrySource>1</odometrySource>
-            <publish_odom_tf>true</publish_odom_tf>
-            <publish_wheel_tf>true</publish_wheel_tf>
-            <odometry_topic>diffdrive/odom</odometry_topic>
-            <odometry_frame>diff_odom</odometry_frame>
-            <robot_base_frame>base_footprint_diff</robot_base_frame>
-        </plugin>
-    </gazebo>
+  <gazebo>
+      <plugin name="gazebo_ros_joint_state_publisher"
+          filename="libgazebo_ros_joint_state_publisher.so">
+          <update_rate>20</update_rate>
+          <joint_name>left_wheel_joint</joint_name>
+          <joint_name>right_wheel_joint</joint_name>
+      </plugin>
+  </gazebo>
+  <gazebo>
+      <plugin filename="libgazebo_ros2_control.so" name="gazebo_ros2_control">
+        <namespace>diffdrive</namespace>
+        <robot_param>robot_description</robot_param>
+        <robot_param_node>robot_state_publisher</robot_param_node>
+        <parameters>$(find coop_robot_bringup)/config/diff_controller.yaml</parameters>
+        <controller_manager_name>controller_manager</controller_manager_name>
+      </plugin>
+  </gazebo>
+  <ros2_control name="GazeboSystem" type="system">
+    <hardware>
+      <plugin>gazebo_ros2_control/GazeboSystem</plugin>
+    </hardware>
+    <joint name="left_wheel_joint">
+      <command_interface name="velocity">
+        <param name="min">-0.5</param>
+        <param name="max">0.5</param>
+      </command_interface>
+      <state_interface name="position"/>
+      <state_interface name="velocity"/>
+    </joint>
+    <joint name="right_wheel_joint">
+      <command_interface name="velocity">
+        <param name="min">-0.5</param>
+        <param name="max">0.5</param>
+      </command_interface>
+      <state_interface name="position"/>
+      <state_interface name="velocity"/>
+    </joint>
+  </ros2_control>
     <gazebo reference="wheel_right">
       <material>Gazebo/Green</material>

File: my_robot_description/urdf/long_pallet.xacro (robot description, xacro)
@@ -15,5 +15,5 @@
         rpy="0 0 0" />
       <mass
-        value="0.1" />
+        value="1" />
       <inertia
         ixx="0.05011773"
@@ -47,21 +47,21 @@
       </geometry>
       <surface>
-        <contact>
-          <poissons_ratio>0.347</poissons_ratio>
-          <elastic_modulus>8.8e+09</elastic_modulus>
-          <ode>
-            <soft_cfm>0.0</soft_cfm>
-            <soft_erp>2e25</soft_erp>
-            <kp>1e15</kp>
-            <kd>1e13</kd>
-            <max_vel>0.01</max_vel>
-            <min_depth>100</min_depth>
-          </ode>
+        <contact friction="0.01">
+        <poissons_ratio>0.347</poissons_ratio>
+        <elastic_modulus>8.8e+09</elastic_modulus>
+        <ode>
+          <soft_cfm>2e+20</soft_cfm>
+          <soft_erp>2e+20</soft_erp>
+          <kp>1</kp>
+          <kd>10</kd>
+          <max_vel>0.01</max_vel>
+          <min_depth>1</min_depth>
+        </ode>
         </contact>
         <friction>
             <fdir1>0 0 0</fdir1>
-            <mu>1</mu>
+            <mu>0.5</mu>
             <slip2>0</slip2>
-            <mu2>1</mu2>
+            <mu2>0.5</mu2>
             <slip1>0</slip1>
         </friction>
