Commit message: add urdf

File: my_robot_description/urdf/diffdrive.xacro (robot description, xacro)
@@ -1,8 +1,7 @@
 <?xml version="1.0"?>
-<robot name="diffdrive" xmlns:xacro="http://www.ros.org/wiki/xacro">
-  <link name="base_footprint">
-  </link>
+<robot xmlns:xacro="http://www.ros.org/wiki/xacro" name="diffdrive" >
+  <link name="base_footprint"></link>
   <joint name="base_link_to_base_footprint" type="fixed">
-    <origin xyz="0 0 0" rpy="0 0 0"/>
+    <origin xyz="0 0 0.05" rpy="0 0 0"/>
     <parent link="base_footprint"/>
     <child link="base_link"/>
@@ -15,5 +14,5 @@
         rpy="0 0 0" />
       <mass
-        value="3.99707593295727" />
+        value="10" />
       <inertia
         ixx="0.0338286081756613"
@@ -30,5 +29,5 @@
       <geometry>
         <mesh
-          filename="package://my_robot_description/meshes/diffdrive_meshes/base_link.STL" />
+          filename="file:///$(find my_robot_description)/meshes/diffdrive_meshes/base_link.STL" />
       </geometry>
       <material
@@ -44,5 +43,5 @@
       <geometry>
         <mesh
-          filename="package://my_robot_description/meshes/diffdrive_meshes/base_link.STL" />
+          filename="file:///$(find my_robot_description)/meshes/diffdrive_meshes/base_link.STL" />
       </geometry>
     </collision>
@@ -70,5 +69,5 @@
       <geometry>
         <mesh
-          filename="package://my_robot_description/meshes/diffdrive_meshes/caster_wheel_01.STL" />
+          filename="file:///$(find my_robot_description)/meshes/diffdrive_meshes/caster_wheel_01.STL"/>
       </geometry>
       <material
@@ -84,5 +83,5 @@
       <geometry>
         <mesh
-          filename="package://my_robot_description/meshes/diffdrive_meshes/caster_wheel_01.STL" />
+          filename="file:///$(find my_robot_description)/meshes/diffdrive_meshes/caster_wheel_01.STL" />
       </geometry>
     </collision>
@@ -123,5 +122,5 @@
       <geometry>
         <mesh
-          filename="package://my_robot_description/meshes/diffdrive_meshes/caster_01.STL" />
+          filename="file:///$(find my_robot_description)/meshes/diffdrive_meshes/caster_01.STL" />
       </geometry>
       <material
@@ -137,5 +136,5 @@
       <geometry>
         <mesh
-          filename="package://my_robot_description/meshes/diffdrive_meshes/caster_01.STL" />
+          filename="file:///$(find my_robot_description)/meshes/diffdrive_meshes/caster_01.STL" />
       </geometry>
     </collision>
@@ -155,5 +154,5 @@
   </joint>
   <link
-    name="caster_wheel_02">/diffdrive
+    name="caster_wheel_02">
     <inertial>
       <origin
@@ -176,5 +175,5 @@
       <geometry>
         <mesh
-          filename="package://my_robot_description/meshes/diffdrive_meshes/caster_wheel_02.STL" />
+          filename="file:///$(find my_robot_description)/meshes/diffdrive_meshes/caster_wheel_02.STL" />
       </geometry>
       <material
@@ -190,5 +189,5 @@
       <geometry>
         <mesh
-          filename="package://my_robot_description/meshes/diffdrive_meshes/caster_wheel_02.STL" />
+          filename="file:///$(find my_robot_description)/meshes/diffdrive_meshes/caster_wheel_02.STL" />
       </geometry>
     </collision>
@@ -229,5 +228,5 @@
       <geometry>
         <mesh
-          filename="package://my_robot_description/meshes/diffdrive_meshes/caster_02.STL" />
+          filename="file:///$(find my_robot_description)/meshes/diffdrive_meshes/caster_02.STL" />
       </geometry>
       <material
@@ -243,5 +242,5 @@
       <geometry>
         <mesh
-          filename="package://my_robot_description/meshes/diffdrive_meshes/caster_02.STL" />
+          filename="file:///$(find my_robot_description)/meshes/diffdrive_meshes/caster_02.STL" />
       </geometry>
     </collision>
@@ -282,5 +281,5 @@
       <geometry>
         <mesh
-          filename="package://my_robot_description/meshes/diffdrive_meshes/caster_wheel_03.STL" />
+          filename="file:///$(find my_robot_description)/meshes/diffdrive_meshes/caster_wheel_03.STL" />
       </geometry>
       <material
@@ -296,5 +295,5 @@
       <geometry>
         <mesh
-          filename="package://my_robot_description/meshes/diffdrive_meshes/caster_wheel_03.STL" />
+          filename="file:///$(find my_robot_description)/meshes/diffdrive_meshes/caster_wheel_03.STL" />
       </geometry>
     </collision>
@@ -335,5 +334,5 @@
       <geometry>
         <mesh
-          filename="package://my_robot_description/meshes/diffdrive_meshes/caster_03.STL" />
+          filename="file:///$(find my_robot_description)/meshes/diffdrive_meshes/caster_03.STL" />
       </geometry>
       <material
@@ -349,5 +348,5 @@
       <geometry>
         <mesh
-          filename="package://my_robot_description/meshes/diffdrive_meshes/caster_03.STL" />
+          filename="file:///$(find my_robot_description)/meshes/diffdrive_meshes/caster_03.STL" />
       </geometry>
     </collision>
@@ -388,5 +387,5 @@
       <geometry>
         <mesh
-          filename="package://my_robot_description/meshes/diffdrive_meshes/caster_wheel_04.STL" />
+          filename="file:///$(find my_robot_description)/meshes/diffdrive_meshes/caster_wheel_04.STL" />
       </geometry>
       <material
@@ -402,5 +401,5 @@
       <geometry>
         <mesh
-          filename="package://my_robot_description/meshes/diffdrive_meshes/caster_wheel_04.STL" />
+          filename="file:///$(find my_robot_description)/meshes/diffdrive_meshes/caster_wheel_04.STL" />
       </geometry>
     </collision>
@@ -441,5 +440,5 @@
       <geometry>
         <mesh
-          filename="package://my_robot_description/meshes/diffdrive_meshes/caster_04.STL" />
+          filename="file:///$(find my_robot_description)/meshes/diffdrive_meshes/caster_04.STL" />
       </geometry>
       <material
@@ -455,5 +454,5 @@
       <geometry>
         <mesh
-          filename="package://my_robot_description/meshes/diffdrive_meshes/caster_04.STL" />
+          filename="file:///$(find my_robot_description)/meshes/diffdrive_meshes/caster_04.STL" />
       </geometry>
     </collision>
@@ -479,5 +478,5 @@
         rpy="0 0 0" />
       <mass
-        value="0.240470068076377" />
+        value="2" />
       <inertia
         ixx="0.000245137261047143"
@@ -494,5 +493,5 @@
       <geometry>
         <mesh
-          filename="package://my_robot_description/meshes/diffdrive_meshes/wheel_01.STL" />
+          filename="file:///$(find my_robot_description)/meshes/diffdrive_meshes/wheel_01.STL" />
       </geometry>
       <material
@@ -508,5 +507,5 @@
       <geometry>
         <mesh
-          filename="package://my_robot_description/meshes/diffdrive_meshes/wheel_01.STL" />
+          filename="file:///$(find my_robot_description)/meshes/diffdrive_meshes/wheel_01.STL" />
       </geometry>
     </collision>
@@ -532,5 +531,5 @@
         rpy="0 0 0" />
       <mass
-        value="0.240470068076377" />
+        value="2" />
       <inertia
         ixx="0.000245137261047143"
@@ -547,5 +546,5 @@
       <geometry>
         <mesh
-          filename="package://my_robot_description/meshes/diffdrive_meshes/wheel_02.STL" />
+          filename="file:///$(find my_robot_description)/meshes/diffdrive_meshes/wheel_02.STL" />
       </geometry>
       <material
@@ -561,5 +560,5 @@
       <geometry>
         <mesh
-          filename="package://my_robot_description/meshes/diffdrive_meshes/wheel_02.STL" />
+          filename="file:///$(find my_robot_description)/meshes/diffdrive_meshes/wheel_02.STL" />
       </geometry>
     </collision>
@@ -590,10 +589,15 @@
             <right_joint>joint_wheel_02</right_joint>
             <!-- kinematics -->
-            <wheel_separation>0.5</wheel_separation>
+            <wheel_separation>0.55</wheel_separation>
             <wheel_diameter>0.12</wheel_diameter>
+            <wheelAcceleration>0.0</wheelAcceleration>
+            <!-- Maximum torque which the wheels can produce, in Nm, defaults to 5 Nm -->
+            <wheelTorque>5</wheelTorque>
             <!-- input -->
             <command_topic>cmd_vel</command_topic>
             <!-- output -->
             <publish_odom>true</publish_odom>
+            <!-- Odometry source, 0 for ENCODER, 1 for WORLD, defaults to WORLD -->
+            <odometrySource>1</odometrySource>
             <publish_odom_tf>true</publish_odom_tf>
             <publish_wheel_tf>true</publish_wheel_tf>

Commit message: update

File: my_robot_description/urdf/diffdrive.xacro (robot description, xacro)
@@ -44,15 +44,12 @@
     <inertial>
       <origin
-        xyz="-0.00843797932248264 7.91524717263514E-05 0.0510944704707574"
-        rpy="0 0 0" />
-      <mass
-        value="5.20115624935193" />
-      <inertia
-        ixx="0.0441950216113175"
-        ixy="-6.1273841754346E-08"
-        ixz="1.5363609769836E-06"
-        iyy="0.0338853571996096"
-        iyz="2.75308042467669E-07"
-        izz="0.077237000418039" />
+        xyz="-0.0244064139228468 -6.45065062421235E-07 0.0569804687199345"
+        rpy="0 0 0" />
+      <mass
+        value="1.66720366185749" />
+      <inertia
+        ixx="0.01" ixy="0.0" ixz="0.0"
+        iyy="0.01" iyz="0.0"
+        izz="0.01"/>
     </inertial>
     <visual>
@@ -78,14 +75,26 @@
           filename="file:///$(find my_robot_description)/meshes/diffdrive_meshes/base_link.STL" />
       </geometry>
-    </collision>
-  </link>
-  <link
-    name="wheel_left">
-    <inertial>
-      <origin
-        xyz="0 0.0257257525083612 -2.77555756156289E-17"
-        rpy="0 0 0" />
-      <mass
-        value="2.40470068076377" />
+     <surface>
+        <poissons_ratio>0.347</poissons_ratio>
+        <elastic_modulus>8.8e+09</elastic_modulus>
+        <ode>
+          <soft_cfm>2e+20</soft_cfm>
+          <soft_erp>2e+40</soft_erp>
+          <kp>1000</kp>
+          <kd>1</kd>
+          <max_vel>0.01</max_vel>
+          <min_depth>1.0</min_depth>
+        </ode>
+      </surface>
+    </collision>
+  </link>
+  <link
+    name="Wheel_left">
+    <inertial>
+      <origin
+        xyz="1.11022302462516E-16 0.0257257525083613 -8.32667268468867E-17"
+        rpy="0 0 0" />
+      <mass
+        value="4.40470068076377" />
       <inertia
         ixx="0.000245137261047142"
@@ -102,15 +111,19 @@
       <geometry>
         <mesh
-          filename="file:///$(find my_robot_description)/meshes/diffdrive_meshes/wheel_left.STL" />
-      </geometry>
-      <material name="wheel" />
-    </visual>
-    <collision>
-      <origin
-        xyz="0 0 0"
-        rpy="0 0 0" />
-      <geometry>
-        <mesh
-          filename="file:///$(find my_robot_description)/meshes/diffdrive_meshes/wheel_left.STL" />
+          filename="file:///$(find my_robot_description)/meshes/diffdrive_meshes/Wheel_left.STL" />
+      </geometry>
+      <material
+        name="">
+        <color
+          rgba="0.792156862745098 0.819607843137255 0.933333333333333 1" />
+      </material>
+    </visual>
+    <collision>
+      <origin
+        xyz="0 0 0"
+        rpy="0 0 0" />
+      <geometry>
+        <mesh
+          filename="file:///$(find my_robot_description)/meshes/diffdrive_meshes/Wheel_left.STL" />
       </geometry>
     </collision>
@@ -125,22 +138,22 @@
       link="base_link_diff" />
     <child
-      link="wheel_left" />
+      link="Wheel_left" />
     <axis
       xyz="0 1 0" />
   </joint>
   <link
-    name="wheel_right">
-    <inertial>
-      <origin
-        xyz="5.55111512312578E-17 0.0257257525083612 5.55111512312578E-17"
-        rpy="0 0 0" />
-      <mass
-        value="2.40470068076377" />
+    name="Wheel_right">
+    <inertial>
+      <origin
+        xyz="-1.38777878078145E-16 0.0257257525084522 5.55111512312578E-17"
+        rpy="0 0 0" />
+      <mass
+        value="4.40470068076377" />
       <inertia
         ixx="0.000245137261047143"
-        ixy="4.26861241081053E-21"
-        ixz="-6.7762635780344E-21"
+        ixy="5.77297627993884E-21"
+        ixz="1.35525271560688E-20"
         iyy="0.000452624182450972"
-        iyz="1.59972478988236E-20"
+        iyz="1.29229555498199E-20"
         izz="0.000245137261047143" />
     </inertial>
@@ -151,15 +164,19 @@
       <geometry>
         <mesh
-          filename="file:///$(find my_robot_description)/meshes/diffdrive_meshes/wheel_right.STL" />
-      </geometry>
-      <material name="wheel" />
-    </visual>
-    <collision>
-      <origin
-        xyz="0 0 0"
-        rpy="0 0 0" />
-      <geometry>
-        <mesh
-          filename="file:///$(find my_robot_description)/meshes/diffdrive_meshes/wheel_right.STL" />
+          filename="file:///$(find my_robot_description)/meshes/diffdrive_meshes/Wheel_right.STL" />
+      </geometry>
+      <material
+        name="">
+        <color
+          rgba="0.792156862745098 0.819607843137255 0.933333333333333 1" />
+      </material>
+    </visual>
+    <collision>
+      <origin
+        xyz="0 0 0"
+        rpy="0 0 0" />
+      <geometry>
+        <mesh
+          filename="file:///$(find my_robot_description)/meshes/diffdrive_meshes/Wheel_right.STL" />
       </geometry>
     </collision>
@@ -174,7 +191,135 @@
       link="base_link_diff" />
     <child
-      link="wheel_right" />
+      link="Wheel_right" />
     <axis
       xyz="0 -1 0" />
+  </joint>
+  <link
+    name="folk_diff_right">
+    <inertial>
+      <origin
+        xyz="0.25796 -0.0675 0.01"
+        rpy="0 0 0" />
+      <mass
+        value="0.052454" />
+      <inertia
+        ixx="4.2123E-05"
+        ixy="1.618E-18"
+        ixz="-1.9029E-14"
+        iyy="0.013244"
+        iyz="2.3396E-16"
+        izz="0.013244" />
+    </inertial>
+    <visual>
+      <origin
+        xyz="0 0 0"
+        rpy="0 0 0" />
+      <geometry>
+        <mesh
+          filename="file:///$(find my_robot_description)/meshes/diffdrive_meshes/folk_right.STL" />
+      </geometry>
+      <material
+        name="">
+        <color
+          rgba="0 1 0 0.5" />
+      </material>
+    </visual>
+    <collision>
+      <origin
+        xyz="0.25796 0.0675 0.01"
+        rpy="0.0 0.0 0.0" />
+        <geometry>
+            <box size="0.55 0.04 0.02"/>
+        </geometry>
+     <surface>
+        <poissons_ratio>0.347</poissons_ratio>
+        <elastic_modulus>8.8e+09</elastic_modulus>
+        <ode>
+          <soft_cfm>2e+20</soft_cfm>
+          <soft_erp>2e+40</soft_erp>
+          <kp>1000</kp>
+          <kd>1</kd>
+          <max_vel>0.01</max_vel>
+          <min_depth>1.0</min_depth>
+        </ode>
+      </surface>
+    </collision>
+  </link>
+  <joint
+    name="folk_diff_right_fixed"
+    type="fixed">
+    <origin
+      xyz="-0.107035355338993 0 0.120000000000272"
+      rpy="0 0 -3.14159265358979" />
+    <parent
+      link="base_link_diff" />
+    <child
+      link="folk_diff_right" />
+    <axis
+      xyz="0 0 0" />
+  </joint>
+  <link
+    name="folk_diff_left">
+    <inertial>
+      <origin
+        xyz="0.25796 0.0675 0.01"
+        rpy="0 0 0" />
+      <mass
+        value="0.052454" />
+      <inertia
+        ixx="4.2123E-05"
+        ixy="1.618E-18"
+        ixz="-1.9029E-14"
+        iyy="0.013244"
+        iyz="2.3396E-16"
+        izz="0.013244" />
+    </inertial>
+    <visual>
+      <origin
+        xyz="0 0 0"
+        rpy="0 0 0" />
+      <geometry>
+        <mesh
+          filename="file:///$(find my_robot_description)/meshes/diffdrive_meshes/folk_left.STL" />
+      </geometry>
+      <material
+        name="">
+        <color
+          rgba="0 0.5 0 0.5" />
+      </material>
+    </visual>
+    <collision>
+      <origin
+        xyz="0.25796 0.0675 0.01"
+        rpy="0.0 0.0 0.0" />
+        <geometry>
+            <box size="0.55 0.04 0.02"/>
+        </geometry>
+     <surface>
+        <poissons_ratio>0.347</poissons_ratio>
+        <elastic_modulus>8.8e+09</elastic_modulus>
+        <ode>
+          <soft_cfm>2e+20</soft_cfm>
+          <soft_erp>2e+40</soft_erp>
+          <kp>1000</kp>
+          <kd>1</kd>
+          <max_vel>0.01</max_vel>
+          <min_depth>1.0</min_depth>
+        </ode>
+      </surface>
+    </collision>
+  </link>
+  <joint
+    name="folk_diff_left_fixed"
+    type="fixed">
+    <origin
+      xyz="-0.107035355338993 0 0.120000000000272"
+      rpy="0 0 -3.14159265358979" />
+    <parent
+      link="base_link_diff" />
+    <child
+      link="folk_diff_left" />
+    <axis
+      xyz="0 0 0" />
   </joint>
     <gazebo>

File: my_robot_description/urdf/diffdrive_control.xacro (robot description, xacro)
@@ -180,4 +180,5 @@
   <gazebo>
       <plugin filename="libgazebo_ros2_control.so" name="gazebo_ros2_control">
+        <namespace>diffdrive</namespace>
         <robot_param>robot_description</robot_param>
         <robot_param_node>robot_state_publisher</robot_param_node>

File: my_robot_description/urdf/long_pallet.xacro (robot description, xacro)
@@ -53,8 +53,8 @@
           <soft_cfm>2e+20</soft_cfm>
           <soft_erp>2e+20</soft_erp>
-          <kp>1</kp>
-          <kd>10</kd>
+          <kp>1000</kp>
+          <kd>1</kd>
           <max_vel>0.01</max_vel>
-          <min_depth>1</min_depth>
+          <min_depth>1.0</min_depth>
         </ode>
         </contact>
