Commit message: add gazebo

File: my_robot_description/urdf/ackermann.xacro (robot description, xacro)
@@ -5,4 +5,10 @@
 <robot
   name="ackermann">
+  <link name="base_footprint"></link>
+  <joint name="base_link_to_base_footprint" type="fixed">
+    <origin xyz="0 0 0.05" rpy="0 0 0"/>
+    <parent link="base_footprint"/>
+    <child link="base_link"/>
+  </joint>
   <link
     name="base_link">
@@ -363,3 +369,43 @@
       xyz="0 1 0" />
   </joint>
+    <gazebo>
+      <plugin name="gazebo_ros_ackermann_drive" filename="libgazebo_ros_ackermann_drive.so">
+        <ros>
+          <namespace>ackermann</namespace>
+          <remapping>cmd_vel:=cmd_vel</remapping>
+          <remapping>odom:=odom</remapping>
+          <remapping>distance:=distance</remapping>
+        </ros>
+        <update_rate>100.0</update_rate>
+        <!-- wheels -->
+        <front_left_joint>Fr_Wheel_R_joint</front_left_joint>
+        <front_right_joint>Fr_Wheel_R_joint</front_right_joint>
+        <rear_left_joint>Bk_Wheel_L_joint</rear_left_joint>
+        <rear_right_joint>Bk_Wheel_R_joint</rear_right_joint>
+        <left_steering_joint>Bk_Turn_L_joint</left_steering_joint>
+        <right_steering_joint>Bk_Turn_R_joint</right_steering_joint>
+        <!-- <steering_wheel_joint>steering_joint</steering_wheel_joint> -->
+        <!-- Max absolute steer angle for tyre in radians-->
+        <!-- Any cmd_vel angular z greater than this would be capped -->
+        <max_steer>0.6458</max_steer>
+        <!-- Max absolute steering angle of steering wheel -->
+        <max_steering_angle>7.85</max_steering_angle>
+        <!-- Max absolute linear speed in m/s -->
+        <max_speed>20</max_speed>
+        <!-- PID tuning -->
+        <left_steering_pid_gain>1500 0 1</left_steering_pid_gain>
+        <left_steering_i_range>0 0</left_steering_i_range>
+        <right_steering_pid_gain>1500 0 1</right_steering_pid_gain>
+        <right_steering_i_range>0 0</right_steering_i_range>
+        <linear_velocity_pid_gain>1000 0 1</linear_velocity_pid_gain>
+        <linear_velocity_i_range>0 0</linear_velocity_i_range>
+        <!-- output -->
+        <publish_odom>true</publish_odom>
+        <publish_odom_tf>true</publish_odom_tf>
+        <publish_wheel_tf>true</publish_wheel_tf>
+        <publish_distance>true</publish_distance>
+        <odometry_frame>odom_demo</odometry_frame>
+        <robot_base_frame>base_link</robot_base_frame>
+      </plugin>
+    </gazebo>
 </robot>

File: my_robot_description/urdf/diffdrive.xacro (robot description, xacro)
@@ -1,9 +1,40 @@
 <?xml version="1.0"?>
-<robot xmlns:xacro="http://www.ros.org/wiki/xacro" name="diffdrive" >
+<robot xmlns:xacro="http://www.ros.org/wiki/xacro" name="diffdrive2" >
+<!-- This URDF was automatically created by SolidWorks to URDF Exporter! Originally created by Stephen Brawner (brawner@gmail.com)
+     Commit Version: 1.6.0-4-g7f85cfe  Build Version: 1.6.7995.38578
+     For more information, please see http://wiki.ros.org/sw_urdf_exporter -->
   <link name="base_footprint"></link>
   <joint name="base_link_to_base_footprint" type="fixed">
-    <origin xyz="0 0 0.05" rpy="0 0 0"/>
+    <origin xyz="0 0 0" rpy="0 0 0"/>
     <parent link="base_footprint"/>
     <child link="base_link"/>
+  </joint>
+  <link name="laser_frame">
+    <visual>
+      <geometry>
+        <cylinder radius="0.05" length="0.04"/>
+      </geometry>
+    </visual>
+    <collision>
+      <geometry>
+        <cylinder radius="0.05" length="0.04"/>
+      </geometry>
+    </collision>
+      <inertial>
+      <origin
+        xyz="0 0 0"
+        rpy="0 0 0" />
+      <mass
+        value="0.1" />
+      <inertia
+        ixx="0.01" ixy="0.0" ixz="0.0"
+        iyy="0.01" iyz="0.0"
+        izz="0.01"/>
+    </inertial>
+  </link>
+  <joint name="laser_joint" type="fixed">
+    <origin xyz="0 0 0.12" rpy="0 0 0"/>
+    <parent link="base_link"/>
+    <child link="laser_frame"/>
   </joint>
   <link
@@ -11,15 +42,15 @@
     <inertial>
       <origin
-        xyz="0.410002757772882 0.223304099954227 0.383656044234519"
-        rpy="0 0 0" />
-      <mass
-        value="10" />
-      <inertia
-        ixx="0.0338286081756613"
-        ixy="2.69812394512863E-07"
-        ixz="6.04312596661445E-10"
-        iyy="0.0771999899846764"
-        iyz="1.18867676606539E-08"
-        izz="0.0441560434041183" />
+        xyz="-0.00843797932248264 7.91524717263514E-05 0.0510944704707574"
+        rpy="0 0 0" />
+      <mass
+        value="4.20115624935193" />
+      <inertia
+        ixx="0.0441950216113175"
+        ixy="-6.1273841754346E-08"
+        ixz="1.5363609769836E-06"
+        iyy="0.0338853571996096"
+        iyz="2.75308042467669E-07"
+        izz="0.077237000418039" />
     </inertial>
     <visual>
@@ -34,5 +65,5 @@
         name="">
         <color
-          rgba="1 1 1 0.4" />
+          rgba="0.752941176470588 0.752941176470588 0.752941176470588 1" />
       </material>
     </visual>
@@ -48,132 +79,26 @@
   </link>
   <link
-    name="caster_wheel_01">
+    name="Wheel_left">
     <inertial>
       <origin
-        xyz="0.00442419024671004 0.0407882700915736 5.11365806366015E-08"
-        rpy="0 0 0" />
-      <mass
-        value="0.0159163609587196" />
-      <inertia
-        ixx="3.04804887255873E-06"
-        ixy="3.8115153686273E-07"
-        ixz="1.01515368617414E-10"
-        iyy="2.55687129048666E-06"
-        iyz="-5.57379950267749E-11"
-        izz="2.82872222947099E-06" />
-    </inertial>
-    <visual>
-      <origin
-        xyz="0 0 0"
-        rpy="0 0 0" />
-      <geometry>
-        <mesh
-          filename="file:///$(find my_robot_description)/meshes/diffdrive_meshes/caster_wheel_01.STL"/>
-      </geometry>
-      <material
-        name="">
-        <color
-          rgba="1 1 1 1" />
-      </material>
-    </visual>
-    <collision>
-      <origin
-        xyz="0 0 0"
-        rpy="0 0 0" />
-      <geometry>
-        <mesh
-          filename="file:///$(find my_robot_description)/meshes/diffdrive_meshes/caster_wheel_01.STL" />
-      </geometry>
-    </collision>
-  </link>
-  <joint
-    name="joint_caster_wheel_01"
-    type="continuous">
-    <origin
-      xyz="0.649922237049609 -0.238297834751047 0.157919253158435"
-      rpy="1.5707963267949 0 -1.55646155726161" />
-    <parent
-      link="base_link" />
-    <child
-      link="caster_wheel_01" />
-    <axis
-      xyz="0 1 0" />
-  </joint>
-  <link
-    name="caster_01">
-    <inertial>
-      <origin
-        xyz="0.0214652433425613 0.00180092427509927 0"
-        rpy="0 0 0" />
-      <mass
-        value="0.0351037181525611" />
-      <inertia
-        ixx="6.69573691459496E-06"
-        ixy="-4.2351647362715E-22"
-        ixz="-1.4756902127946E-20"
-        iyy="6.69573691459495E-06"
-        iyz="-1.46444055646388E-20"
-        izz="1.13592998252083E-05" />
-    </inertial>
-    <visual>
-      <origin
-        xyz="0 0 0"
-        rpy="0 0 0" />
-      <geometry>
-        <mesh
-          filename="file:///$(find my_robot_description)/meshes/diffdrive_meshes/caster_01.STL" />
-      </geometry>
-      <material
-        name="">
-        <color
-          rgba="0.250980392156863 0.250980392156863 0.250980392156863 1" />
-      </material>
-    </visual>
-    <collision>
-      <origin
-        xyz="0 0 0"
-        rpy="0 0 0" />
-      <geometry>
-        <mesh
-          filename="file:///$(find my_robot_description)/meshes/diffdrive_meshes/caster_01.STL" />
-      </geometry>
-    </collision>
-  </link>
-  <joint
-    name="joint_caster_01"
-    type="continuous">
-    <origin
-      xyz="0 0 0"
-      rpy="0 0 0.296802859073811" />
-    <parent
-      link="caster_wheel_01" />
-    <child
-      link="caster_01" />
-    <axis
-      xyz="0.292464356117457 0.956276424681065 0" />
-  </joint>
-  <link
-    name="caster_wheel_02">
-    <inertial>
-      <origin
-        xyz="-0.00376546230151442 0.0407882700171175 -0.00232266139324588"
-        rpy="0 0 0" />
-      <mass
-        value="0.0159163608550056" />
-      <inertia
-        ixx="2.98751038693051E-06"
-        ixy="-3.24432619179736E-07"
-        ixz="9.80449894252071E-08"
-        iyy="2.55687121621709E-06"
-        iyz="-2.00049983095585E-07"
-        izz="2.88926070956337E-06" />
-    </inertial>
-    <visual>
-      <origin
-        xyz="0 0 0"
-        rpy="0 0 0" />
-      <geometry>
-        <mesh
-          filename="file:///$(find my_robot_description)/meshes/diffdrive_meshes/caster_wheel_02.STL" />
+        xyz="0 0.0257257525083612 -2.77555756156289E-17"
+        rpy="0 0 0" />
+      <mass
+        value="0.240470068076377" />
+      <inertia
+        ixx="0.000245137261047142"
+        ixy="5.12745004835681E-20"
+        ixz="0"
+        iyy="0.000452624182450971"
+        iyz="-5.57841424911612E-20"
+        izz="0.000245137261047142" />
+    </inertial>
+    <visual>
+      <origin
+        xyz="0 0 0"
+        rpy="0 0 0" />
+      <geometry>
+        <mesh
+          filename="file:///$(find my_robot_description)/meshes/diffdrive_meshes/Wheel_left.STL" />
       </geometry>
       <material
@@ -189,294 +114,29 @@
       <geometry>
         <mesh
-          filename="file:///$(find my_robot_description)/meshes/diffdrive_meshes/caster_wheel_02.STL" />
+          filename="file:///$(find my_robot_description)/meshes/diffdrive_meshes/Wheel_left.STL" />
       </geometry>
     </collision>
   </link>
   <joint
-    name="joint_caster_wheel_02"
+    name="right_wheel_joint"
     type="continuous">
     <origin
-      xyz="0.649922237049609 -0.548297834751047 0.157919253158437"
-      rpy="1.5707963267949 0 2.14107688053925" />
+      xyz="-0.000999999999839296 -0.249999999999933 0.0305000000006919"
+      rpy="0 0.774914173734372 3.14159265358979" />
     <parent
       link="base_link" />
     <child
-      link="caster_wheel_02" />
+      link="Wheel_left" />
     <axis
-      xyz="0 1 0" />
+      xyz="0 -1 0" />
   </joint>
   <link
-    name="caster_02">
+    name="Wheel_right">
     <inertial>
       <origin
-        xyz="0.0214652433425611 0.00180092427509934 1.11022302462516E-16"
-        rpy="0 0 0" />
-      <mass
-        value="0.0351037181525611" />
-      <inertia
-        ixx="6.69573691459496E-06"
-        ixy="3.17637355220363E-22"
-        ixz="2.2446373102239E-20"
-        iyy="6.69573691459495E-06"
-        iyz="-2.1572870375383E-21"
-        izz="1.13592998252083E-05" />
-    </inertial>
-    <visual>
-      <origin
-        xyz="0 0 0"
-        rpy="0 0 0" />
-      <geometry>
-        <mesh
-          filename="file:///$(find my_robot_description)/meshes/diffdrive_meshes/caster_02.STL" />
-      </geometry>
-      <material
-        name="">
-        <color
-          rgba="0.250980392156863 0.250980392156863 0.250980392156863 1" />
-      </material>
-    </visual>
-    <collision>
-      <origin
-        xyz="0 0 0"
-        rpy="0 0 0" />
-      <geometry>
-        <mesh
-          filename="file:///$(find my_robot_description)/meshes/diffdrive_meshes/caster_02.STL" />
-      </geometry>
-    </collision>
-  </link>
-  <joint
-    name="joint_caster_02"
-    type="continuous">
-    <origin
-      xyz="0 0 0"
-      rpy="2.96311522163044 0.525941308677483 2.79662415169577" />
-    <parent
-      link="caster_wheel_02" />
-    <child
-      link="caster_02" />
-    <axis
-      xyz="0.292464356117457 0.956276424681065 0" />
-  </joint>
-  <link
-    name="caster_wheel_03">
-    <inertial>
-      <origin
-        xyz="-0.00376546080228934 0.0407882711178764 -0.00232265994952238"
-        rpy="0 0 0" />
-      <mass
-        value="0.0159163611002415" />
-      <inertia
-        ixx="2.98751079488814E-06"
-        ixy="-3.24432397210381E-07"
-        ixz="9.8043942933475E-08"
-        iyy="2.55687160406272E-06"
-        iyz="-2.0005032862318E-07"
-        izz="2.88926023574823E-06" />
-    </inertial>
-    <visual>
-      <origin
-        xyz="0 0 0"
-        rpy="0 0 0" />
-      <geometry>
-        <mesh
-          filename="file:///$(find my_robot_description)/meshes/diffdrive_meshes/caster_wheel_03.STL" />
-      </geometry>
-      <material
-        name="">
-        <color
-          rgba="0.792156862745098 0.819607843137255 0.933333333333333 1" />
-      </material>
-    </visual>
-    <collision>
-      <origin
-        xyz="0 0 0"
-        rpy="0 0 0" />
-      <geometry>
-        <mesh
-          filename="file:///$(find my_robot_description)/meshes/diffdrive_meshes/caster_wheel_03.STL" />
-      </geometry>
-    </collision>
-  </link>
-  <joint
-    name="joint_caster_wheel_03"
-    type="continuous">
-    <origin
-      xyz="0.169922237049587 -0.548297834751047 0.157919253158437"
-      rpy="1.5707963267949 0 2.11677958982226" />
-    <parent
-      link="base_link" />
-    <child
-      link="caster_wheel_03" />
-    <axis
-      xyz="0 1 0" />
-  </joint>
-  <link
-    name="caster_03">
-    <inertial>
-      <origin
-        xyz="0.0214652433425609 0.00180092427509926 1.11022302462516E-16"
-        rpy="0 0 0" />
-      <mass
-        value="0.0351037181525611" />
-      <inertia
-        ixx="6.69573691459494E-06"
-        ixy="3.17637355220363E-22"
-        ixz="8.37106779903664E-22"
-        iyy="6.69573691459494E-06"
-        iyz="-3.25743725223382E-21"
-        izz="1.13592998252082E-05" />
-    </inertial>
-    <visual>
-      <origin
-        xyz="0 0 0"
-        rpy="0 0 0" />
-      <geometry>
-        <mesh
-          filename="file:///$(find my_robot_description)/meshes/diffdrive_meshes/caster_03.STL" />
-      </geometry>
-      <material
-        name="">
-        <color
-          rgba="0.250980392156863 0.250980392156863 0.250980392156863 1" />
-      </material>
-    </visual>
-    <collision>
-      <origin
-        xyz="0 0 0"
-        rpy="0 0 0" />
-      <geometry>
-        <mesh
-          filename="file:///$(find my_robot_description)/meshes/diffdrive_meshes/caster_03.STL" />
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