Commit message: add gazebo

File: my_robot_description/urdf/mecanum.xacro (robot description, xacro)
@@ -1,23 +1,52 @@
-<?xml version="1.0" encoding="utf-8"?>
-<!-- This URDF was automatically created by SolidWorks to URDF Exporter! Originally created by Stephen Brawner (brawner@gmail.com)
-     Commit Version: 1.6.0-4-g7f85cfe  Build Version: 1.6.7995.38578
-     For more information, please see http://wiki.ros.org/sw_urdf_exporter -->
-<robot
-  name="mecanum">
+<?xml version="1.0"?>
+<robot xmlns:xacro="http://www.ros.org/wiki/xacro" name="mecanum" >
+  <link name="base_footprint"></link>
+  <joint name="base_link_to_base_footprint" type="fixed">
+    <origin xyz="0 0 0.11" rpy="0 0 1.57"/>
+    <parent link="base_footprint"/>
+    <child link="base_link"/>
+    <dynamics damping="0" friction="0.00001"/>
+  </joint>
+  <link name="laser_frame">
+    <visual>
+      <geometry>
+        <cylinder radius="0.05" length="0.04"/>
+      </geometry>
+    </visual>
+    <collision>
+      <geometry>
+        <cylinder radius="0.05" length="0.04"/>
+      </geometry>
+    </collision>
+      <inertial>
+      <origin
+        xyz="0 0 0"
+        rpy="0 0 0" />
+      <mass
+        value="0.1" />
+      <inertia
+        ixx="0.01" ixy="0.0" ixz="0.0"
+        iyy="0.01" iyz="0.0"
+        izz="0.01"/>
+    </inertial>
+  </link>
+  <joint name="laser_joint" type="fixed">
+    <origin xyz="0 0 0.02" rpy="0 0 0"/>
+    <parent link="base_link"/>
+    <child link="laser_frame"/>
+    <dynamics damping="0" friction="0.00001"/>
+  </joint>
   <link
     name="base_link">
     <inertial>
       <origin
-        xyz="0.351806015356857 0.274861498867373 0.395577155294245"
-        rpy="0 0 0" />
-      <mass
-        value="2.0229199501028" />
-      <inertia
-        ixx="0.0130277088512019"
-        ixy="2.84366610936317E-08"
-        ixz="-6.62413626810912E-20"
-        iyy="0.0427706330641988"
-        iyz="5.3832707352464E-16"
-        izz="0.0299520637832313" />
+        xyz="-1.14613076807046E-08 -4.91918539569092E-07 -0.0135289818533382"
+        rpy="0 0 0" />
+      <mass
+        value="2" />
+      <inertia
+        ixx="0.01" ixy="0.0" ixz="0.0"
+        iyy="0.01" iyz="0.0"
+        izz="0.01"/>
     </inertial>
     <visual>
@@ -46,26 +75,23 @@
   </link>
   <link
-    name="Wheel_01">
-    <inertial>
-      <origin
-        xyz="-0.00910192948839045 0.0203724822485673 -0.0223132954397111"
-        rpy="0 0 0" />
-      <mass
-        value="0.199180638989129" />
-      <inertia
-        ixx="0.000106836233715406"
-        ixy="2.35922457854813E-06"
-        ixz="-2.58397942811303E-06"
-        iyy="0.000102609720496205"
-        iyz="5.78361709963215E-06"
-        izz="0.000101555676344914" />
-    </inertial>
-    <visual>
-      <origin
-        xyz="0 0 0"
-        rpy="0 0 0" />
-      <geometry>
-        <mesh
-          filename="file:///$(find my_robot_description)/meshes/mecanum_meshes/Wheel_01.STL" />
+    name="wheel_fr_right">
+    <inertial>
+      <origin
+        xyz="0.0194370630585373 -0.0176353488184189 0.00817275304865103"
+        rpy="0 0 0" />
+      <mass
+        value="0.0002" />
+      <inertia
+        ixx="0.01" ixy="0.0" ixz="0.0"
+        iyy="0.01" iyz="0.0"
+        izz="0.01"/>
+    </inertial>
+    <visual>
+      <origin
+        xyz="0 0 0"
+        rpy="0 0 0" />
+      <geometry>
+        <mesh
+          filename="file:///$(find my_robot_description)/meshes/mecanum_meshes/wheel_fr_right.STL" />
       </geometry>
       <material
@@ -81,2723 +107,225 @@
       <geometry>
         <mesh
-          filename="file:///$(find my_robot_description)/meshes/mecanum_meshes/Wheel_01.STL" />
+          filename="file:///$(find my_robot_description)/meshes/mecanum_meshes/wheel_fr_right.STL" />
       </geometry>
     </collision>
   </link>
   <joint
-    name="wheel_J1_joint"
-    type="continuous">
+    name="joint_fr_right"
+    type="fixed">
     <origin
-      xyz="0.169305469629096 -0.538072117578766 0.235572147509167"
-      rpy="-1.35872938250007 1.21658582746707 0.981977586530455" />
+      xyz="0.196431540449915 0.18250000000009 -0.0500000000000465"
+      rpy="2.56826265176299 -0.701812030330357 2.7542816171153" />
     <parent
       link="base_link" />
     <child
-      link="Wheel_01" />
+      link="wheel_fr_right" />
     <axis
-      xyz="0.288439512685233 -0.645602546092763 0.707106781186863" />
-  </joint>
-  <link
-    name="Wheel01_ball01">
-    <inertial>
-      <origin
-        xyz="-0.0402740558208334 -0.0418043308783602 -0.0194356671750471"
-        rpy="0 0 0" />
-      <mass
-        value="0.0137538624053492" />
-      <inertia
-        ixx="2.72479617507416E-06"
-        ixy="-1.58818677610181E-22"
-        ixz="1.74700545371199E-21"
-        iyy="2.72479617507411E-06"
-        iyz="-1.73377056391115E-21"
-        izz="6.02477450305521E-07" />
-    </inertial>
-    <visual>
-      <origin
-        xyz="0 0 0"
-        rpy="0 0 0" />
-      <geometry>
-        <mesh
-          filename="file:///$(find my_robot_description)/meshes/mecanum_meshes/Wheel01_ball01.STL" />
-      </geometry>
-      <material
-        name="">
-        <color
-          rgba="0.298039215686275 0.298039215686275 0.298039215686275 1" />
-      </material>
-    </visual>
-    <collision>
-      <origin
-        xyz="0 0 0"
-        rpy="0 0 0" />
-      <geometry>
-        <mesh
-          filename="file:///$(find my_robot_description)/meshes/mecanum_meshes/Wheel01_ball01.STL" />
+      xyz="0.707106781183754 -0.64156167526822 0.297319048886856" />
+    <dynamics damping="0" friction="0.00001"/>
+  </joint>
+  <link
+    name="wheel_bk_right">
+    <inertial>
+      <origin
+        xyz="0.0194370630585368 -0.017635348818419 0.00817275304865139"
+        rpy="0 0 0" />
+      <mass
+        value="0.0002" />
+      <inertia
+        ixx="0.01" ixy="0.0" ixz="0.0"
+        iyy="0.01" iyz="0.0"
+        izz="0.01"/>
+    </inertial>
+    <visual>
+      <origin
+        xyz="0 0 0"
+        rpy="0 0 0" />
+      <geometry>
+        <mesh
+          filename="file:///$(find my_robot_description)/meshes/mecanum_meshes/wheel_bk_right.STL" />
+      </geometry>
+      <material
+        name="">
+        <color
+          rgba="0.776470588235294 0.756862745098039 0.737254901960784 1" />
+      </material>
+    </visual>
+    <collision>
+      <origin
+        xyz="0 0 0"
+        rpy="0 0 0" />
+      <geometry>
+        <mesh
+          filename="file:///$(find my_robot_description)/meshes/mecanum_meshes/wheel_bk_right.STL" />
       </geometry>
     </collision>
   </link>
   <joint
-    name="Wheel01_ball01_joint"
-    type="continuous">
+    name="joint_bk_right"
+    type="fixed">
     <origin
-      xyz="0.0819035958512037 -0.183321520420573 0.200785903047669"
-      rpy="-3.14159265358979 0 1.56562261314474" />
-    <parent
-      link="Wheel_01" />
-    <child
-      link="Wheel01_ball01" />
-    <axis
-      xyz="0.644101608802806 -0.291775800122612 0.707106781186863" />
-  </joint>
-  <link
-    name="Wheel01_ball02">
-    <inertial>
-      <origin
-        xyz="-0.0402740558207703 -0.0418043308785501 -0.0194356671747692"
-        rpy="0 0 0" />
-      <mass
-        value="0.0137538624053494" />
-      <inertia
-        ixx="2.72479617507474E-06"
-        ixy="-5.29395592033938E-23"
-        ixz="-7.18770983216318E-18"
-        iyy="2.72479617507474E-06"
-        iyz="-7.18522167288062E-18"
-        izz="6.02477450306733E-07" />
-    </inertial>
-    <visual>
-      <origin
-        xyz="0 0 0"
-        rpy="0 0 0" />
-      <geometry>
-        <mesh
-          filename="file:///$(find my_robot_description)/meshes/mecanum_meshes/Wheel01_ball02.STL" />
-      </geometry>
-      <material
-        name="">
-        <color
-          rgba="0.298039215686275 0.298039215686275 0.298039215686275 1" />
-      </material>
-    </visual>
-    <collision>
-      <origin
-        xyz="0 0 0"
-        rpy="0 0 0" />
-      <geometry>
-        <mesh
-          filename="file:///$(find my_robot_description)/meshes/mecanum_meshes/Wheel01_ball02.STL" />
-      </geometry>
-    </collision>
-  </link>
-  <joint
-    name="Wheel01_ball02_joint"
-    type="continuous">
-    <origin
-      xyz="0.0819035958512037 -0.183321520420573 0.200785903047669"
-      rpy="2.78299843386616 -0.0849715703112149 1.9555303213579" />
-    <parent
-      link="Wheel_01" />
-    <child
-      link="Wheel01_ball02" />
-    <axis
-      xyz="0.644101608804425 -0.291775800118351 0.707106781187146" />
-  </joint>
-  <link
-    name="Wheel01_ball03">
-    <inertial>
-      <origin
-        xyz="-0.0402740558207018 -0.041804330878756 -0.0194356671744681"
-        rpy="0 0 0" />
-      <mass
-        value="0.0137538624053492" />
-      <inertia
-        ixx="2.7247961750741E-06"
-        ixy="0"
-        ixz="-1.49742190184759E-17"
-        iyy="2.7247961750741E-06"
-        iyz="-1.49760454332685E-17"
-        izz="6.0247745030547E-07" />
-    </inertial>
-    <visual>
-      <origin
-        xyz="0 0 0"
-        rpy="0 0 0" />
-      <geometry>
-        <mesh
-          filename="file:///$(find my_robot_description)/meshes/mecanum_meshes/Wheel01_ball03.STL" />
-      </geometry>
-      <material
-        name="">
-        <color
-          rgba="0.298039215686275 0.298039215686275 0.298039215686275 1" />
-      </material>
-    </visual>
-    <collision>
-      <origin
-        xyz="0 0 0"
-        rpy="0 0 0" />
-      <geometry>
-        <mesh
-          filename="file:///$(find my_robot_description)/meshes/mecanum_meshes/Wheel01_ball03.STL" />
-      </geometry>
-    </collision>
-  </link>
-  <joint
-    name="Wheel01_ball03_joint"
-    type="continuous">
-    <origin
-      xyz="0.0819035958512037 -0.183321520420573 0.200785903047669"
-      rpy="2.41921187729642 -0.0249635401401731 2.3502466957237" />
-    <parent
-      link="Wheel_01" />
-    <child
-      link="Wheel01_ball03" />
-    <axis
-      xyz="0.644101608806368 -0.291775800114774 0.707106781186852" />
-  </joint>
-  <link
-    name="Wheel01_ball04">
-    <inertial>
-      <origin
-        xyz="-0.0402740558206848 -0.0418043308788076 -0.0194356671743925"
-        rpy="0 0 0" />
-      <mass
-        value="0.0137538624053492" />
-      <inertia
-        ixx="2.72479617507479E-06"
-        ixy="5.29395592033938E-23"
-        ixz="-1.69269740690319E-17"
-        iyy="2.72479617507479E-06"
-        iyz="-1.69235462325735E-17"
-        izz="6.02477450306836E-07" />
-    </inertial>
-    <visual>
-      <origin
-        xyz="0 0 0"
-        rpy="0 0 0" />
-      <geometry>
-        <mesh
-          filename="file:///$(find my_robot_description)/meshes/mecanum_meshes/Wheel01_ball04.STL" />
-      </geometry>
-      <material
-        name="">
-        <color
-          rgba="0.298039215686275 0.298039215686275 0.298039215686275 1" />
-      </material>
-    </visual>
-    <collision>
-      <origin
-        xyz="0 0 0"
-        rpy="0 0 0" />
-      <geometry>
-        <mesh
-          filename="file:///$(find my_robot_description)/meshes/mecanum_meshes/Wheel01_ball04.STL" />
-      </geometry>
-    </collision>
-  </link>
-  <joint
-    name="Wheel01_ball04_joint"
-    type="continuous">
-    <origin
-      xyz="0.0819035958512037 -0.183321520420573 0.200785903047669"
-      rpy="2.10230543117965 0.16441253380222 2.70238074706886" />
-    <parent
-      link="Wheel_01" />
-    <child
-      link="Wheel01_ball04" />
-    <axis
-      xyz="0.644101608806124 -0.291775800115496 0.707106781186777" />
-  </joint>
-  <link
-    name="Wheel01_ball05">
-    <inertial>
-      <origin
-        xyz="-0.0402740558206904 -0.0418043308787904 -0.0194356671744176"
-        rpy="0 0 0" />
-      <mass
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