Commit message: spawn bot

File: my_robot_description/urdf/ackermann.xacro (robot description, xacro)
@@ -1,29 +1,23 @@
-<?xml version="1.0" encoding="utf-8"?>
-<!-- This URDF was automatically created by SolidWorks to URDF Exporter! Originally created by Stephen Brawner (brawner@gmail.com)
-     Commit Version: 1.6.0-4-g7f85cfe  Build Version: 1.6.7995.38578
-     For more information, please see http://wiki.ros.org/sw_urdf_exporter -->
-<robot
-  name="ackermann">
-  <link name="base_footprint"></link>
-  <joint name="base_link_to_base_footprint" type="fixed">
-    <origin xyz="0 0 0.05" rpy="0 0 0"/>
-    <parent link="base_footprint"/>
-    <child link="base_link"/>
-  </joint>
-  <link
-    name="base_link">
-    <inertial>
-      <origin
-        xyz="0.401114315271127 -0.448682126989679 0.224781274259531"
-        rpy="0 0 0" />
-      <mass
-        value="3.65693181713568" />
-      <inertia
-        ixx="0.015169090067713"
-        ixy="1.82796488685576E-07"
-        ixz="-1.05010040455871E-07"
-        iyy="0.0313226511863623"
-        iyz="3.45960820674392E-07"
-        izz="0.0456140714001489" />
+<?xml version="1.0"?>
+<robot xmlns:xacro="http://www.ros.org/wiki/xacro" name="ackermann" >
+  <link name="base_footprint_ack">
+  </link>
+  <joint name="base_link_ack_to_base_footprint_ack" type="fixed">
+    <origin xyz="0 0 0.12" rpy="0 0 1.57"/>
+    <parent link="base_footprint_ack"/>
+    <child link="base_link_ack"/>
+  </joint>
+  <link
+    name="base_link_ack">
+    <inertial>
+      <origin
+        xyz="-4.21303280262464E-07 -0.0595327816236317 -0.0394837308817142"
+        rpy="0 0 0" />
+      <mass
+        value="1" />
+      <inertia
+        ixx="0.01" ixy="0.0" ixz="0.0"
+        iyy="0.01" iyz="0.0"
+        izz="0.01"/>
     </inertial>
     <visual>
@@ -38,5 +32,5 @@
         name="">
         <color
-          rgba="0.898039215686275 0.917647058823529 0.929411764705882 1" />
+          rgba="1 1 1 0.4" />
       </material>
     </visual>
@@ -52,26 +46,223 @@
   </link>
   <link
-    name="Bk_Turn_R">
-    <inertial>
-      <origin
-        xyz="-0.00706815393332894 -0.0356877943586188 -0.0125569877404127"
-        rpy="0 0 0" />
-      <mass
-        value="0.0449308336357259" />
-      <inertia
-        ixx="1.53282078261686E-05"
-        ixy="2.85913088017762E-06"
-        ixz="2.99325552978407E-06"
-        iyy="2.1535058174114E-05"
-        iyz="7.01449169886432E-07"
-        izz="1.46105917335225E-05" />
-    </inertial>
-    <visual>
-      <origin
-        xyz="0 0 0"
-        rpy="0 0 0" />
-      <geometry>
-        <mesh
-          filename="file:///$(find my_robot_description)/meshes/ackermann_meshes/Bk_Turn_R.STL" />
+    name="front_left">
+    <inertial>
+      <origin
+        xyz="9.4647E-14 -0.015274 3.8664E-14"
+        rpy="0 0 0" />
+      <mass
+        value="0.2" />
+      <inertia
+        ixx="0.01" ixy="0.0" ixz="0.0"
+        iyy="0.01" iyz="0.0"
+        izz="0.01"/>
+    </inertial>
+    <visual>
+      <origin
+        xyz="0 0 0"
+        rpy="0 0 0" />
+      <geometry>
+        <mesh
+          filename="file:///$(find my_robot_description)/meshes/ackermann_meshes/front_left.STL" />
+      </geometry>
+      <material
+        name="">
+        <color
+          rgba="0 1 0 0.5" />
+      </material>
+    </visual>
+    <collision>
+      <origin
+        xyz="0 0 0"
+        rpy="0 0 0" />
+      <geometry>
+        <mesh
+          filename="file:///$(find my_robot_description)/meshes/ackermann_meshes/front_left.STL" />
+      </geometry>
+    </collision>
+  </link>
+  <joint
+    name="front_left_joint"
+    type="continuous">
+    <origin
+      xyz="-0.301000000000045 0.0190000000000679 -0.0695000000000887"
+      rpy="3.14159265358979 0.0849179307157281 -1.5707963267949" />
+    <parent
+      link="base_link_ack" />
+    <child
+      link="front_left" />
+    <axis
+      xyz="0 -1 0" />
+  </joint>
+  <link
+    name="front_right">
+    <inertial>
+      <origin
+        xyz="-9.9698E-14 0.025726 -2.2427E-14"
+        rpy="0 0 0" />
+      <mass
+        value="0.2" />
+      <inertia
+        ixx="0.01" ixy="0.0" ixz="0.0"
+        iyy="0.01" iyz="0.0"
+        izz="0.01"/>
+    </inertial>
+    <visual>
+      <origin
+        xyz="0 0 0"
+        rpy="0 0 0" />
+      <geometry>
+        <mesh
+          filename="file:///$(find my_robot_description)/meshes/ackermann_meshes/front_right.STL" />
+      </geometry>
+      <material
+        name="">
+        <color
+          rgba="0 1 0 0.5" />
+      </material>
+    </visual>
+    <collision>
+      <origin
+        xyz="0 0 0"
+        rpy="0 0 0" />
+      <geometry>
+        <mesh
+          filename="file:///$(find my_robot_description)/meshes/ackermann_meshes/front_right.STL" />
+      </geometry>
+    </collision>
+  </link>
+  <joint
+    name="front_right_joint"
+    type="continuous">
+    <origin
+      xyz="0.259999999999977 0.0190000000000679 -0.0695000000000887"
+      rpy="3.14159265358979 -0.692237011731428 1.5707963267949" />
+    <parent
+      link="base_link_ack" />
+    <child
+      link="front_right" />
+    <axis
+      xyz="0 1 0" />
+  </joint>
+  <link
+    name="left_steering">
+    <inertial>
+      <origin
+        xyz="0.013865 -0.0153 -0.021185"
+        rpy="0 0 0" />
+      <mass
+        value="0.2" />
+      <inertia
+        ixx="0.01" ixy="0.0" ixz="0.0"
+        iyy="0.01" iyz="0.0"
+        izz="0.01"/>
+    </inertial>
+    <visual>
+      <origin
+        xyz="0 0 0"
+        rpy="0 0 0" />
+      <geometry>
+        <mesh
+          filename="file:///$(find my_robot_description)/meshes/ackermann_meshes/left_steering.STL" />
+      </geometry>
+      <material
+        name="">
+        <color
+          rgba="0.79216 0.81961 0.93333 1" />
+      </material>
+    </visual>
+    <collision>
+      <origin
+        xyz="0 0 0"
+        rpy="0 0 0" />
+      <geometry>
+        <mesh
+          filename="file:///$(find my_robot_description)/meshes/ackermann_meshes/left_steering.STL" />
+      </geometry>
+    </collision>
+  </link>
+  <joint
+    name="left_steering_joint"
+    type="continuous">
+    <origin
+      xyz="-0.229999999999977 -0.544750000000063 -0.0837500000002837"
+      rpy="3.14159265358979 0 1.56870378020951" />
+    <parent
+      link="base_link_ack" />
+    <child
+      link="left_steering" />
+    <axis
+      xyz="0 0 1" />
+  </joint>
+  <link
+    name="rear_left">
+    <inertial>
+      <origin
+        xyz="-3.3074E-13 0.025977 4.563E-14"
+        rpy="0 0 0" />
+      <mass
+        value="0.2" />
+      <inertia
+        ixx="0.01" ixy="0.0" ixz="0.0"
+        iyy="0.01" iyz="0.0"
+        izz="0.01"/>
+    </inertial>
+    <visual>
+      <origin
+        xyz="0 0 0"
+        rpy="0 0 0" />
+      <geometry>
+        <mesh
+          filename="file:///$(find my_robot_description)/meshes/ackermann_meshes/rear_left.STL" />
+      </geometry>
+      <material
+        name="">
+        <color
+          rgba="0 1 0 0.5" />
+      </material>
+    </visual>
+    <collision>
+      <origin
+        xyz="0 0 0"
+        rpy="0 0 0" />
+      <geometry>
+        <mesh
+          filename="file:///$(find my_robot_description)/meshes/ackermann_meshes/rear_left.STL" />
+      </geometry>
+    </collision>
+  </link>
+  <joint
+    name="rear_left_joint"
+    type="continuous">
+    <origin
+      xyz="0 -0.0367488381424265 -0.0159999999999999"
+      rpy="3.14159265358979 1.57056930363849 0" />
+    <parent
+      link="left_steering" />
+    <child
+      link="rear_left" />
+    <axis
+      xyz="0 1 0" />
+  </joint>
+  <link
+    name="right_steering">
+    <inertial>
+      <origin
+        xyz="-0.0138648135893726 -0.0152975648321685 -0.0211847288398291"
+        rpy="0 0 0" />
+      <mass
+        value="0.202056975407" />
+      <inertia
+        ixx="0.01" ixy="0.0" ixz="0.0"
+        iyy="0.01" iyz="0.0"
+        izz="0.01"/>
+    </inertial>
+    <visual>
+      <origin
+        xyz="0 0 0"
+        rpy="0 0 0" />
+      <geometry>
+        <mesh
+          filename="file:///$(find my_robot_description)/meshes/ackermann_meshes/right_steering.STL" />
       </geometry>
       <material
@@ -87,325 +278,114 @@
       <geometry>
         <mesh
-          filename="file:///$(find my_robot_description)/meshes/ackermann_meshes/Bk_Turn_R.STL" />
-      </geometry>
-    </collision>
-  </link>
-  <joint
-    name="Bk_Turn_R_joint"
-    type="continuous">
-    <origin
-      xyz="0.614114914635943 -0.813820257624567 0.180513128382613"
-      rpy="-1.5707963267949 0 2.56288301873173" />
-    <parent
-      link="base_link" />
-    <child
-      link="Bk_Turn_R" />
+          filename="file:///$(find my_robot_description)/meshes/ackermann_meshes/right_steering.STL" />
+      </geometry>
+    </collision>
+  </link>
+  <joint
+    name="right_steering_joint"
+    type="continuous">
+    <origin
+      xyz="0.230000000000023 -0.544750000000063 -0.0837500000002836"
+      rpy="3.14159265358979 0 -1.56162994548732" />
+    <parent
+      link="base_link_ack" />
+    <child
+      link="right_steering" />
+    <axis
+      xyz="0 0 1" />
+  </joint>
+  <link
+    name="rear_right">
+    <inertial>
+      <origin
+        xyz="3.3534E-13 0.025722 -9.3148E-14"
+        rpy="0 0 0" />
+      <mass
+        value="0.2" />
+      <inertia
+        ixx="0.01" ixy="0.0" ixz="0.0"
+        iyy="0.01" iyz="0.0"
+        izz="0.01"/>
+    </inertial>
+    <visual>
+      <origin
+        xyz="0 0 0"
+        rpy="0 0 0" />
+      <geometry>
+        <mesh
+          filename="file:///$(find my_robot_description)/meshes/ackermann_meshes/rear_right.STL" />
+      </geometry>
+      <material
+        name="">
+        <color
+          rgba="0 1 0 0.5" />
+      </material>
+    </visual>
+    <collision>
+      <origin
+        xyz="0 0 0"
+        rpy="0 0 0" />
+      <geometry>
+        <mesh
+          filename="file:///$(find my_robot_description)/meshes/ackermann_meshes/rear_right.STL" />
+      </geometry>
+    </collision>
+  </link>
+  <joint
+    name="rear_right_joint"
+    type="continuous">
+    <origin
+      xyz="0 -0.0370034448281129 -0.0159999999999995"
+      rpy="3.14159265358979 -1.55976234848309 0" />
+    <parent
+      link="right_steering" />
+    <child
+      link="rear_right" />
     <axis
       xyz="0 1 0" />
   </joint>
-  <link
-    name="Bk_Wheel_R">
-    <inertial>
-      <origin
-        xyz="-2.77555756156289E-17 0.0504681649917319 5.55111512312578E-16"
-        rpy="0 0 0" />
-      <mass
-        value="0.244535505413318" />
-      <inertia
-        ixx="0.000245434009544367"
-        ixy="3.23675773692E-21"
-        ixz="9.52912065661088E-22"
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
File: my_robot_description/urdf/diffdrive.xacro (robot description, xacro)
@@ -1,7 +1,9 @@
 <?xml version="1.0"?>
-<robot xmlns:xacro="http://www.ros.org/wiki/xacro" name="diffdrive2" >
+<robot xmlns:xacro="http://www.ros.org/wiki/xacro" name="diffdrive" >
 <!-- This URDF was automatically created by SolidWorks to URDF Exporter! Originally created by Stephen Brawner (brawner@gmail.com)
      Commit Version: 1.6.0-4-g7f85cfe  Build Version: 1.6.7995.38578
      For more information, please see http://wiki.ros.org/sw_urdf_exporter -->
+  <material name="wheel">
+    <color rgba="0 1 0 0.5" /> </material>
   <link name="base_footprint"></link>
   <joint name="base_link_to_base_footprint" type="fixed">
@@ -79,5 +81,5 @@
   </link>
   <link
-    name="Wheel_left">
+    name="wheel_left">
     <inertial>
       <origin
@@ -100,19 +102,15 @@
       <geometry>
         <mesh
-          filename="file:///$(find my_robot_description)/meshes/diffdrive_meshes/Wheel_left.STL" />
-      </geometry>
-      <material
-        name="">
-        <color
-          rgba="0.792156862745098 0.819607843137255 0.933333333333333 1" />
-      </material>
-    </visual>
-    <collision>
-      <origin
-        xyz="0 0 0"
-        rpy="0 0 0" />
-      <geometry>
-        <mesh
-          filename="file:///$(find my_robot_description)/meshes/diffdrive_meshes/Wheel_left.STL" />
+          filename="file:///$(find my_robot_description)/meshes/diffdrive_meshes/wheel_left.STL" />
+      </geometry>
+      <material name="wheel" />
+    </visual>
+    <collision>
+      <origin
+        xyz="0 0 0"
+        rpy="0 0 0" />
+      <geometry>
+        <mesh
+          filename="file:///$(find my_robot_description)/meshes/diffdrive_meshes/wheel_left.STL" />
       </geometry>
     </collision>
@@ -127,10 +125,10 @@
       link="base_link" />
     <child
-      link="Wheel_left" />
+      link="wheel_left" />
     <axis
       xyz="0 -1 0" />
   </joint>
   <link
-    name="Wheel_right">
+    name="wheel_right">
     <inertial>
       <origin
@@ -153,19 +151,15 @@
       <geometry>
         <mesh
-          filename="file:///$(find my_robot_description)/meshes/diffdrive_meshes/Wheel_right.STL" />
-      </geometry>
-      <material
-        name="">
-        <color
-          rgba="0.792156862745098 0.819607843137255 0.933333333333333 1" />
-      </material>
-    </visual>
-    <collision>
-      <origin
-        xyz="0 0 0"
-        rpy="0 0 0" />
-      <geometry>
-        <mesh
-          filename="file:///$(find my_robot_description)/meshes/diffdrive_meshes/Wheel_right.STL" />
+          filename="file:///$(find my_robot_description)/meshes/diffdrive_meshes/wheel_right.STL" />
+      </geometry>
+      <material name="wheel" />
+    </visual>
+    <collision>
+      <origin
+        xyz="0 0 0"
+        rpy="0 0 0" />
+      <geometry>
+        <mesh
+          filename="file:///$(find my_robot_description)/meshes/diffdrive_meshes/wheel_right.STL" />
       </geometry>
     </collision>
@@ -180,5 +174,5 @@
       link="base_link" />
     <child
-      link="Wheel_right" />
+      link="wheel_right" />
     <axis
       xyz="0 1 0" />
@@ -215,5 +209,5 @@
         <sensor name="laser" type="ray">
             <pose> 0 0 0 0 0 0 </pose>
-            <visualize>true</visualize>
+            <visualize>false</visualize>
             <update_rate>10</update_rate>
             <ray>

File: my_robot_description/urdf/mecanum.xacro (robot description, xacro)
@@ -1,12 +1,12 @@
 <?xml version="1.0"?>
 <robot xmlns:xacro="http://www.ros.org/wiki/xacro" name="mecanum" >
-  <link name="base_footprint"></link>
-  <joint name="base_link_to_base_footprint" type="fixed">
-    <origin xyz="0 0 0.11" rpy="0 0 1.57"/>
-    <parent link="base_footprint"/>
-    <child link="base_link"/>
-    <dynamics damping="0" friction="0.00001"/>
-  </joint>
-  <link name="laser_frame">
+  <link name="base_footprint_mec">
+  </link>
+  <joint name="base_link_mec_to_base_footprint_mec" type="fixed">
+    <origin xyz="0 0 0.12" rpy="0 0 1.57"/>
+    <parent link="base_footprint_mec"/>
+    <child link="base_link_mec"/>
+  </joint>
+  <link name="laser_mec">
     <visual>
       <geometry>
@@ -19,10 +19,10 @@
       </geometry>
     </collision>
-      <inertial>
-      <origin
-        xyz="0 0 0"
-        rpy="0 0 0" />
-      <mass
-        value="0.1" />
+    <inertial>
+      <origin
+        xyz="0 0 0"
+        rpy="0 0 0" />
+      <mass
+        value="0.01" />
       <inertia
         ixx="0.01" ixy="0.0" ixz="0.0"
@@ -33,10 +33,9 @@
   <joint name="laser_joint" type="fixed">
     <origin xyz="0 0 0.02" rpy="0 0 0"/>
-    <parent link="base_link"/>
-    <child link="laser_frame"/>
-    <dynamics damping="0" friction="0.00001"/>
-  </joint>
-  <link
-    name="base_link">
+    <parent link="base_link_mec"/>
+    <child link="laser_mec"/>
+  </joint>
+  <link
+    name="base_link_mec">
     <inertial>
       <origin
@@ -44,5 +43,5 @@
         rpy="0 0 0" />
       <mass
-        value="2" />
+        value="1" />
       <inertia
         ixx="0.01" ixy="0.0" ixz="0.0"
@@ -106,6 +105,5 @@
         rpy="0 0 0" />
       <geometry>
-        <mesh
-          filename="file:///$(find my_robot_description)/meshes/mecanum_meshes/wheel_fr_right.STL" />
+        <cylinder radius="0.07" length="0.04" />
       </geometry>
     </collision>
@@ -118,10 +116,9 @@
       rpy="2.56826265176299 -0.701812030330357 2.7542816171153" />
     <parent
-      link="base_link" />
+      link="base_link_mec" />
     <child
       link="wheel_fr_right" />
     <axis
       xyz="0.707106781183754 -0.64156167526822 0.297319048886856" />
-    <dynamics damping="0" friction="0.00001"/>
   </joint>
   <link
@@ -157,6 +154,5 @@
         rpy="0 0 0" />
       <geometry>
-        <mesh
-          filename="file:///$(find my_robot_description)/meshes/mecanum_meshes/wheel_bk_right.STL" />
+        <cylinder radius="0.07" length="0.04" />
       </geometry>
     </collision>
@@ -169,10 +165,9 @@
       rpy="2.56826265176299 -0.701812030330358 2.7542816171153" />
     <parent
-      link="base_link" />
+      link="base_link_mec" />
     <child
       link="wheel_bk_right" />
     <axis
       xyz="0.707106781183753 -0.641561675268222 0.297319048886854" />
-    <dynamics damping="0" friction="0.00001"/>
   </joint>
   <link
@@ -208,6 +203,5 @@
         rpy="0 0 0" />
       <geometry>
-        <mesh
-          filename="file:///$(find my_robot_description)/meshes/mecanum_meshes/wheel_fr_left.STL" />
+        <cylinder radius="0.07" length="0.04" />
       </geometry>
     </collision>
@@ -220,10 +214,9 @@
       rpy="2.56826265176299 -0.701812030330358 2.7542816171153" />
     <parent
-      link="base_link" />
+      link="base_link_mec" />
     <child
       link="wheel_fr_left" />
     <axis
       xyz="0.707106781183754 -0.641561675268221 0.297319048886855" />
-    <dynamics damping="0" friction="0.00001"/>
   </joint>
   <link
@@ -259,6 +252,5 @@
         rpy="0 0 0" />
       <geometry>
-        <mesh
-          filename="file:///$(find my_robot_description)/meshes/mecanum_meshes/wheel_bk_left.STL" />
+        <cylinder radius="0.07" length="0.04" />
       </geometry>
     </collision>
@@ -271,61 +263,61 @@
       rpy="2.56826265176298 -0.701812030330358 2.7542816171153" />
     <parent
-      link="base_link" />
+      link="base_link_mec" />
     <child
       link="wheel_bk_left" />
     <axis
       xyz="0.707106781183753 -0.641561675268222 0.297319048886854" />
-    <dynamics damping="0" friction="0.00001"/>
   </joint>
 <gazebo>
-<plugin name="gazebo_ros_planar_move" filename="libgazebo_ros_planar_move.so">
-  <ros>
-    <!-- Add a namespace -->
-    <namespace>mec</namespace>
-    <!-- Remap the default topic -->
-    <remapping>cmd_vel:=cmd_vel</remapping>
-    <remapping>odom:=odom</remapping>
-  </ros>
-  <update_rate>100</update_rate>
-  <publish_rate>10</publish_rate>
-  <!-- output -->
-  <publish_odom>true</publish_odom>
-  <publish_odom_tf>true</publish_odom_tf>
-  <odometry_frame>mec_odom</odometry_frame>
-  <robot_base_frame>base_footprint</robot_base_frame>
-  <publish_wheel_tf>true</publish_wheel_tf>
-  <covariance_x>0.0001</covariance_x>
-  <covariance_y>0.0001</covariance_y>
-  <covariance_yaw>0.01</covariance_yaw>
-</plugin>
+  <plugin name="gazebo_ros_planar_move" filename="libgazebo_ros_planar_move.so">
+    <ros>
+      <!-- Add a namespace -->
+      <namespace>mec</namespace>
+      <!-- Remap the default topic -->
+      <remapping>/mec/cmd_vel:=/mec/cmd_vel</remapping>
+      <remapping>odom:=odom</remapping>
+    </ros>
+    <update_rate>100</update_rate>
+    <publish_rate>10</publish_rate>
+    <!-- output -->
+    <publish_odom>true</publish_odom>
+    <publish_odom_tf>true</publish_odom_tf>
+    <odometry_frame>mec_odom</odometry_frame>
+    <robot_base_frame>base_footprint_mec</robot_base_frame>
+    <publish_wheel_tf>true</publish_wheel_tf>
+    <covariance_x>0.0001</covariance_x>
+    <covariance_y>0.0001</covariance_y>
+    <covariance_yaw>0.01</covariance_yaw>
+  </plugin>
 </gazebo>
-    <gazebo reference="laser_frame">
-        <material>Gazebo/Red</material>
-        <sensor name="laser" type="ray">
-            <pose> 0 0 0 0 0 0 </pose>
-            <visualize>false</visualize>
-            <update_rate>10</update_rate>
-            <ray>
-                <scan>
-                    <horizontal>
-                        <samples>360</samples>
-                        <min_angle>-3.14</min_angle>
-                        <max_angle>3.14</max_angle>
-                    </horizontal>
-                </scan>
-                <range>
-                    <min>0.3</min>
-                    <max>12</max>
-                </range>
-            </ray>
-            <plugin name="laser_mec" filename="libgazebo_ros_ray_sensor.so">
-                <namespace>mec</namespace>
-                <ros>
-                    <argument>/out:=scan</argument>
-                </ros>
-                <output_type>sensor_msgs/LaserScan</output_type>
-                <frame_name>laser_frame</frame_name>
-            </plugin>
-        </sensor>
-    </gazebo>
+  <gazebo reference="laser_mec">
+    <material>Gazebo/Red</material>
+    <sensor name="laser" type="ray">
+      <namespace>mec</namespace>
+      <pose>0 0 0 0 0 0</pose>
+      <visualize>false</visualize>
+      <update_rate>10</update_rate>
+      <ray>
+        <scan>
+          <horizontal>
+            <samples>360</samples>
+            <min_angle>-3.14</min_angle>
+            <max_angle>3.14</max_angle>
+          </horizontal>
+        </scan>
+        <range>
+          <min>0.3</min>
+          <max>12</max>
+        </range>
+      </ray>
+      <plugin name="laser_mec" filename="libgazebo_ros_ray_sensor.so">
+        <namespace>mec</namespace>
+        <ros>
+          <argument>/mec/out:=/scan_mec</argument>
+        </ros>
+        <output_type>sensor_msgs/LaserScan</output_type>
+        <frame_name>laser_mec</frame_name>
+      </plugin>
+    </sensor>
+  </gazebo>
 </robot>
