Commit message: formation controller mecanum tuning

File: my_robot_description/urdf/ackermann.xacro (robot description, xacro)
@@ -124,9 +124,8 @@
     <collision>
       <origin
-        xyz="0 0 0"
-        rpy="0 0 0" />
-      <geometry>
-        <mesh
-          filename="file:///$(find my_robot_description)/meshes/ackermann_meshes/front_right.STL" />
+        xyz="0 0.02 0"
+        rpy="1.57 0 0" />
+      <geometry>
+        <cylinder radius="0.06" length="0.02" />
       </geometry>
     </collision>
@@ -184,5 +183,5 @@
   <joint
     name="left_steering_joint"
-    type="continuous">
+    type="revolute">
     <origin
       xyz="-0.229999999999977 -0.544750000000063 -0.0837500000002837"
@@ -194,4 +193,10 @@
     <axis
       xyz="0 0 1" />
+    <limit
+      lower="-1.570796"
+      upper="1.570796"
+      effort="100"
+      velocity="10"
+    />
   </joint>
   <link
@@ -224,9 +229,8 @@
     <collision>
       <origin
-        xyz="0 0 0"
-        rpy="0 0 0" />
-      <geometry>
-        <mesh
-          filename="file:///$(find my_robot_description)/meshes/ackermann_meshes/rear_left.STL" />
+        xyz="0 0.02 0"
+        rpy="1.57 0 0" />
+      <geometry>
+        <cylinder radius="0.06" length="0.02" />
       </geometry>
     </collision>
@@ -283,15 +287,21 @@
   </link>
   <joint
-    name="right_steering_joint"
-    type="continuous">
-    <origin
-      xyz="0.230000000000023 -0.544750000000063 -0.0837500000002836"
-      rpy="3.14159265358979 0 -1.56162994548732" />
-    <parent
-      link="base_link_ack" />
-    <child
-      link="right_steering" />
-    <axis
-      xyz="0 0 1" />
+      name="right_steering_joint"
+      type="revolute">
+      <origin
+        xyz="0.230000000000023 -0.544750000000063 -0.0837500000002836"
+        rpy="3.14159265358979 0 -1.56162994548732" />
+      <parent
+        link="base_link_ack" />
+      <child
+        link="right_steering" />
+      <axis
+        xyz="0 0 1" />
+      <limit
+        lower="-1.570796"
+        upper="1.570796"
+        effort="100"
+        velocity="10"
+      />
   </joint>
   <link
@@ -324,9 +334,8 @@
     <collision>
       <origin
-        xyz="0 0 0"
-        rpy="0 0 0" />
-      <geometry>
-        <mesh
-          filename="file:///$(find my_robot_description)/meshes/ackermann_meshes/rear_right.STL" />
+        xyz="0 0.02 0"
+        rpy="1.57 0 0" />
+      <geometry>
+        <cylinder radius="0.06" length="0.02" />
       </geometry>
     </collision>
@@ -359,4 +368,5 @@
       <rear_left_joint>front_right_joint</rear_left_joint>
       <rear_right_joint>front_left_joint</rear_right_joint>
+      <!-- wheels -->
       <!-- <front_left_joint>front_left_joint</front_left_joint>
       <front_right_joint>front_right_joint</front_right_joint>
@@ -364,6 +374,6 @@
       <rear_right_joint>rear_right_joint</rear_right_joint> -->
       <!-- steering joints -->
-      <left_steering_joint>left_steering_joint</left_steering_joint>
-      <right_steering_joint>right_steering_joint</right_steering_joint>
+      <left_steering_joint>right_steering_joint</left_steering_joint>
+      <right_steering_joint>left_steering_joint</right_steering_joint>
       <!-- Max absolute steer angle for tyre in radians-->
       <!-- Any cmd_vel angular z greater than this would be capped -->

File: my_robot_description/urdf/long_pallet.xacro (robot description, xacro)
@@ -22,5 +22,5 @@
       <geometry>
         <mesh
-          filename="package://my_robot_description/meshes/long_pallet.stl">
+          filename="file:///$(find my_robot_description)/meshes/long_pallet.stl">
         </mesh>
       </geometry>
@@ -37,5 +37,5 @@
       <geometry>
         <mesh
-          filename="package://my_robot_description/meshes/long_pallet.stl">
+          filename="file:///$(find my_robot_description)/meshes/long_pallet.stl">
         </mesh>
       </geometry>

File: my_robot_description/urdf/mecanum.xacro (robot description, xacro)
@@ -4,5 +4,5 @@
   </link>
   <joint name="base_link_mec_to_base_footprint_mec" type="fixed">
-    <origin xyz="0 0 0.12" rpy="0 0 1.57"/>
+    <origin xyz="0 0 0.12" rpy="0 0 -1.57"/>
     <parent link="base_footprint_mec"/>
     <child link="base_link_mec"/>
@@ -43,5 +43,5 @@
         rpy="0 0 0" />
       <mass
-        value="1" />
+        value="0.5" />
       <inertia
         ixx="0.01" ixy="0.0" ixz="0.0"
@@ -275,5 +275,5 @@
       <namespace>mec</namespace>
       <!-- Remap the default topic -->
-      <remapping>/mec/cmd_vel:=/mec/cmd_vel</remapping>
+      <remapping>/mec/cmd_vel:=/cmd_vel_follower</remapping>
       <remapping>odom:=odom</remapping>
     </ros>

Commit message: update result

File: my_robot_description/urdf/ackermann.xacro (robot description, xacro)
@@ -1,26 +1,57 @@
 <?xml version="1.0"?>
 <robot xmlns:xacro="http://www.ros.org/wiki/xacro" name="ackermann" >
-  <link name="base_footprint_ack">
-  </link>
-  <joint name="base_link_ack_to_base_footprint_ack" type="fixed">
+<!-- This URDF was automatically created by SolidWorks to URDF Exporter! Originally created by Stephen Brawner (brawner@gmail.com)
+     Commit Version: 1.6.0-4-g7f85cfe  Build Version: 1.6.7995.38578
+     For more information, please see http://wiki.ros.org/sw_urdf_exporter -->
+  <link name="base_footprint">
+  </link>
+  <joint name="base_link_to_base_footprint" type="fixed">
     <origin xyz="0 0 0.12" rpy="0 0 0"/>
-    <parent link="base_footprint_ack"/>
+    <parent link="base_footprint"/>
     <child link="base_link"/>
   </joint>
+    <link name="laser_frame">
+    <visual>
+      <geometry>
+        <cylinder radius="0.05" length="0.04"/>
+      </geometry>
+    </visual>
+    <collision>
+      <geometry>
+        <cylinder radius="0.05" length="0.04"/>
+      </geometry>
+    </collision>
+    <inertial>
+      <origin
+        xyz="0 0 0"
+        rpy="0 0 0" />
+      <mass
+        value="0.01" />
+      <inertia
+        ixx="0.01" ixy="0.0" ixz="0.0"
+        iyy="0.01" iyz="0.0"
+        izz="0.01"/>
+    </inertial>
+  </link>
+  <joint name="laser_joint" type="fixed">
+    <origin xyz="0 0 0.16" rpy="0 0 0"/>
+    <parent link="base_link"/>
+    <child link="laser_frame"/>
+  </joint>
   <link
     name="base_link">
     <inertial>
       <origin
-        xyz="-0.0651994405179663 4.22434509872449E-07 -0.0239634712761258"
-        rpy="0 0 0" />
-      <mass
-        value="1.25555128497609" />
-      <inertia
-        ixx="0.0414328478617682"
-        ixy="-1.82796488685318E-07"
-        ixz="3.45960820664179E-07"
-        iyy="0.0417152661425413"
-        iyz="1.05010040923958E-07"
-        izz="0.0821338918053197" />
+        xyz="0.377672365616106 0.191340904613787 0.361389269217461"
+        rpy="0 0 0" />
+      <mass
+        value="10.49814568283799" />
+      <inertia
+        ixx="0.0181839157074767"
+        ixy="-7.37148197622945E-07"
+        ixz="-1.13302958356861E-05"
+        iyy="0.0490501696015112"
+        iyz="1.27098343080043E-07"
+        izz="0.0326062941739465" />
     </inertial>
     <visual>
@@ -35,5 +66,5 @@
         name="">
         <color
-          rgba="1 1 1 0.4" />
+          rgba="0.898039215686275 0.917647058823529 0.929411764705882 1" />
       </material>
     </visual>
@@ -49,18 +80,124 @@
   </link>
   <link
+    name="back_left">
+    <inertial>
+      <origin
+        xyz="1.11022302462516E-16 0.0257257517276274 -5.55111512312578E-17"
+        rpy="0 0 0" />
+      <mass
+        value="20" />
+      <inertia
+        ixx="0.000245137261047143"
+        ixy="4.2881704699239E-19"
+        ixz="-6.7762635780344E-20"
+        iyy="0.000452624182450972"
+        iyz="-2.39038653415574E-20"
+        izz="0.000245137261047143" />
+    </inertial>
+    <visual>
+      <origin
+        xyz="0 0 0"
+        rpy="0 0 0" />
+      <geometry>
+        <mesh
+          filename="file:///$(find my_robot_description)/meshes/ackermann_meshes/back_left.STL" />
+      </geometry>
+      <material
+        name="">
+        <color
+          rgba="0.792156862745098 0.819607843137255 0.933333333333333 1" />
+      </material>
+    </visual>
+    <collision>
+      <origin
+        xyz="0 0 0"
+        rpy="0 0 0" />
+      <geometry>
+        <mesh
+          filename="file:///$(find my_robot_description)/meshes/ackermann_meshes/back_left.STL" />
+      </geometry>
+    </collision>
+  </link>
+  <joint
+    name="back_left_joint"
+    type="fixed">
+    <origin
+      xyz="-0.472974166233064 0.26150000012373 -0.0700000000003574"
+      rpy="0 -0.499103249142133 0.000137993798726114" />
+    <parent
+      link="base_link" />
+    <child
+      link="back_left" />
+    <axis
+      xyz="0 1 0" />
+  </joint>
+  <link
+    name="back_right">
+    <inertial>
+      <origin
+        xyz="-1.10100817352077E-12 0.0271271666381976 -4.34874358745674E-13"
+        rpy="0 0 0" />
+      <mass
+        value="20" />
+      <inertia
+        ixx="0.000245137261047142"
+        ixy="-1.61493650009258E-15"
+        ixz="6.7762635780344E-21"
+        iyy="0.000452624182450971"
+        iyz="-6.37965575295475E-16"
+        izz="0.000245137261047143" />
+    </inertial>
+    <visual>
+      <origin
+        xyz="0 0 0"
+        rpy="0 0 0" />
+      <geometry>
+        <mesh
+          filename="file:///$(find my_robot_description)/meshes/ackermann_meshes/back_right.STL" />
+      </geometry>
+      <material
+        name="">
+        <color
+          rgba="0.792156862745098 0.819607843137255 0.933333333333333 1" />
+      </material>
+    </visual>
+    <collision>
+      <origin
+        xyz="0 0 0"
+        rpy="0 0 0" />
+      <geometry>
+        <mesh
+          filename="file:///$(find my_robot_description)/meshes/ackermann_meshes/back_right.STL" />
+      </geometry>
+    </collision>
+  </link>
+  <joint
+    name="back_right_joint"
+    type="fixed">
+    <origin
+      xyz="-0.473573116541797 -0.259095847310483 -0.0700000000003103"
+      rpy="0 0.376238226393869 3.13259128041529" />
+    <parent
+      link="base_link" />
+    <child
+      link="back_right" />
+    <axis
+      xyz="0 1 0" />
+  </joint>
+  <link
     name="front_left">
     <inertial>
       <origin
-        xyz="3.8858E-15 -0.015274 4.6435E-14"
-        rpy="0 0 0" />
-      <mass
-        value="0.24047" />
-      <inertia
-        ixx="0.00024514"
-        ixy="5.4339E-21"
-        ixz="-6.7763E-21"
-        iyy="0.00045262"
-        iyz="6.4709E-20"
-        izz="0.00024514" />
+        xyz="5.55111512312578E-17 0.0257257525083612 2.77555756156289E-17"
+        rpy="0 0 0" />
+      <mass
+        value="2.4" />
+      <inertia
+        ixx="0.000245137261047143"
+        ixy="1.80227445983964E-20"
+        ixz="0"
+        iyy="0.000452624182450971"
+        iyz="4.41329424203013E-20"
+        izz="0.000245137261047143" />
     </inertial>
     <visual>
@@ -75,5 +212,5 @@
         name="">
         <color
-          rgba="0 1 0 0.5" />
+          rgba="0.792156862745098 0.819607843137255 0.933333333333333 1" />
       </material>
     </visual>
@@ -90,8 +227,8 @@
   <joint
     name="front_left_joint"
-    type="continuous">
-    <origin
-      xyz="0.0190000000000679 0.301000000000045 -0.0695000000000887"
-      rpy="3.14159265358979 0.0849179307157281 3.14159265358979" />
+    type="fixed">
+    <origin
+      xyz="-0.00396464466087482 0.250000000000023 -0.0695000000001352"
+      rpy="3.14159265358979 0.391796412189509 3.14159265358979" />
     <parent
       link="base_link" />
@@ -105,15 +242,15 @@
     <inertial>
       <origin
-        xyz="-2.9643E-14 0.025726 3.5749E-14"
-        rpy="0 0 0" />
-      <mass
-        value="0.24047" />
-      <inertia
-        ixx="0.00024514"
-        ixy="5.2554E-21"
+        xyz="-1.2490009027033E-16 0.0257257525083613 -5.55111512312578E-17"
+        rpy="0 0 0" />
+      <mass
+        value="2.4" />
+      <inertia
+        ixx="0.000245137261047143"
+        ixy="-1.9265269650864E-20"
         ixz="0"
-        iyy="0.00045262"
-        iyz="4.3994E-20"
-        izz="0.00024514" />
+        iyy="0.000452624182450972"
+        iyz="-4.3727623063712E-20"
+        izz="0.000245137261047143" />
     </inertial>
     <visual>
@@ -128,5 +265,5 @@
         name="">
         <color
-          rgba="0 1 0 0.5" />
+          rgba="0.792156862745098 0.819607843137255 0.933333333333333 1" />
       </material>
     </visual>
@@ -143,8 +280,8 @@
   <joint
     name="front_right_joint"
-    type="continuous">
-    <origin
-      xyz="0.0190000000000679 -0.259999999999977 -0.0695000000000887"
-      rpy="3.14159265358979 -0.692237011731428 0" />
+    type="fixed">
+    <origin
+      xyz="-0.00396464466092106 -0.250000000000023 -0.0695000000001819"
+      rpy="0 0.467678189791487 3.14159265358979" />
     <parent
       link="base_link" />
@@ -155,259 +292,201 @@
   </joint>
   <link
-    name="left_steering">
-    <inertial>
-      <origin
-        xyz="0.0121532099874294 -0.0166916241895938 -0.0211847288398316"
-        rpy="0 0 0" />
-      <mass
-        value="0.0405602056975407" />
-      <inertia
-        ixx="1.43958495481578E-05"
-        ixy="-1.73339990683825E-06"
-        ixz="-7.11935154287877E-06"
-        iyy="2.95171085845272E-05"
-        iyz="2.08772590818048E-06"
-        izz="3.10994722329793E-05" />
-    </inertial>
-    <visual>
-      <origin
-        xyz="0 0 0"
-        rpy="0 0 0" />
-      <geometry>
-        <mesh
-          filename="file:///$(find my_robot_description)/meshes/ackermann_meshes/left_steering.STL" />
-      </geometry>
-      <material
-        name="">
-        <color
-          rgba="0.792156862745098 0.819607843137255 0.933333333333333 1" />
-      </material>
-    </visual>
-    <collision>
-      <origin
-        xyz="0 0 0"
-        rpy="0 0 0" />
-      <geometry>
-        <mesh
-          filename="file:///$(find my_robot_description)/meshes/ackermann_meshes/left_steering.STL" />
-      </geometry>
-    </collision>
-  </link>
-  <joint
-    name="left_steering_joint"
-    type="continuous">
-    <origin
-      xyz="-0.544750000000063 0.229999999999977 -0.0837500000002837"
-      rpy="3.14159265358979 0 -0.00209254658538632" />
-    <parent
-      link="base_link" />
-    <child
-      link="left_steering" />
-    <axis
-      xyz="0 0 1" />
-  </joint>
-  <link
-    name="rear_left">
-    <inertial>
-      <origin
-        xyz="-1.5192E-06 0.025619 0.006692"
-        rpy="0 0 0" />
-      <mass
-        value="0.24047" />
-      <inertia
-        ixx="0.00024514"
-        ixy="-4.9967E-09"
-        ixz="-5.3615E-10"
-        iyy="0.00045026"
-        iyz="2.201E-05"
-        izz="0.0002475" />
-    </inertial>
-    <visual>
-      <origin
-        xyz="0 0 0"
-        rpy="0 0 0" />
-      <geometry>
-        <mesh
-          filename="file:///$(find my_robot_description)/meshes/ackermann_meshes/rear_left.STL" />
-      </geometry>
-      <material
-        name="">
-        <color
-          rgba="0 1 0 0.5" />
-      </material>
-    </visual>
-    <collision>
-      <origin
-        xyz="0 0 0"
-        rpy="0 0 0" />
-      <geometry>
-        <mesh
-          filename="file:///$(find my_robot_description)/meshes/ackermann_meshes/rear_left.STL" />
-      </geometry>
-    </collision>
-  </link>
-  <joint
-    name="rear_left_joint"
-    type="continuous">
-    <origin
-      xyz="0 -0.0367488381424265 -0.0159999999999999"
-      rpy="3.14159265358979 1.57056930363849 0" />
-    <parent
-      link="left_steering" />
-    <child
-      link="rear_left" />
-    <axis
-      xyz="0 1 0" />
-  </joint>
-  <link
-    name="right_steering">
-    <inertial>
-      <origin
-        xyz="-0.0138648104691156 -0.0152975676601856 -0.021184728839829"
-        rpy="0 0 0" />
-      <mass
-        value="0.0405602056975408" />
-      <inertia
-        ixx="1.49389187707206E-05"
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
File: my_robot_description/urdf/diffdrive.xacro (robot description, xacro)
@@ -116,5 +116,5 @@
         name="">
         <color
-          rgba="0.792156862745098 0.819607843137255 0.933333333333333 1" />
+          rgba="0.898039215686275 0.917647058823529 0.929411764705882 1" />
       </material>
     </visual>
@@ -169,5 +169,5 @@
         name="">
         <color
-          rgba="0.792156862745098 0.819607843137255 0.933333333333333 1" />
+          rgba="0.898039215686275 0.917647058823529 0.929411764705882 1" />
       </material>
     </visual>
@@ -222,5 +222,5 @@
         name="">
         <color
-          rgba="0 1 0 0.5" />
+          rgba="0.898039215686275 0.917647058823529 0.929411764705882 1" />
       </material>
     </visual>
@@ -286,5 +286,5 @@
         name="">
         <color
-          rgba="0 0.5 0 0.5" />
+          rgba="0.898039215686275 0.917647058823529 0.929411764705882 1" />
       </material>
     </visual>
