Commit message: update urdf mec

File: my_robot_description/urdf/mecanum_fork.xacro (robot description, xacro)
@@ -32,5 +32,5 @@
   </link>
   <joint name="laser_joint" type="fixed">
-    <origin xyz="0 0 0.02" rpy="0 0 0"/>
+    <origin xyz="0 0 0.13" rpy="0 0 0"/>
     <parent link="base_link_mec"/>
     <child link="laser_mec"/>

Commit message: update arduino

File: my_robot_description/urdf/mecanum_fork.xacro (robot description, xacro)
@@ -32,5 +32,5 @@
   </link>
   <joint name="laser_joint" type="fixed">
-    <origin xyz="0 0 0.13" rpy="0 0 0"/>
+    <origin xyz="0 0 0.1" rpy="0 0 0"/>
     <parent link="base_link_mec"/>
     <child link="laser_mec"/>
